File: hardware/01_input.kicad_sch (KiCad schematic)
At the start: 19 parts, among them J1 USB4105-GF-A, U1 CH224K, U2 TPS26600PWPR

Commit message: Refine USB-C PD input safety review and validate unrouted KiCad prototype
Parts:
- removed D2: Schottky 1A 40V, symbol BigModular:Device_D_Schottky
- D1: NOTE 12V standoff; 13.3..14.7V breakdown; 19.9V specified pulse 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 -> 12V standoff: sustained 15/20V is a TVS/fuse fault, NOT qua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
- R1: value 1k 1% -> 1k 1% >=0.5W; footprint Resistor_SMD:R_0603_1608Metric -> Resistor_SMD:R_2010_5025Metric; NOTE (none) -> CH224K supply resistor: at 21V fault, VDD>=2.4V, 1% low R, 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
- U2: NOTE MODE to RTN = current-limit auto-retry. SHDN internally pul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 -> Specified reverse-current blocking replaces series diode. M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
Connections:
- net INPUT_SAFE is gone; now on net VBUS_FUSED: C2.1, JP1.1 (A), R6.1, U2.1 (IN), U2.2 (IN)
Other:
- note added: "9 V request only. No USB data. CH224K Rd must be verified on unpowered attach. JP1 OPEN = OFF (default). Close ONLY for an approved dedicated source. PG is diagnostic, not a current-contract detector. No series diode: TPS26600 reverse-current blocking is specified; qualify dead-battery/backfeed on hardware. All bulk capacitance is behind the eFuse. No legacy-host enumeration or CC-current decodin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"
- note removed: "9 V request only. No USB data. CH224K internal Rd: no parallel 5.1k resistors. JP1 OPEN = OFF (default). Close ONLY for an approved dedicated source. PG is diagnostic, not a current-contract detector. All bulk capacitance is behind the eFuse. No legacy-host enumeration or CC-current decoding is implemented."

Commit message: Remove unsafe input TVS and document unqualified surge protection
Parts:
- removed D1: SMBJ12CA, symbol BigModular:Device_D_TVS
- C2: NOTE (none) -> TPS26600 local bypass only. Not an ESD/surge clamp; effecti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
- F1: NOTE Candidate rating, NOT USB current authorization or coordina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 -> Unselected candidate: 32V rating covers steady 20/21V only;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
Other:
- note added: "D1 SMBJ12CA REMOVED: it can burn at sustained 15/20 V. F1 (500 mA / 32 V) is NOT a coordinated surge fuse. TPS26600 OVP (~10.8 V) disconnects OUTPUT, not upstream VBUS. No qualified VBUS transient protection. 9 V request only. No USB data. CH224K Rd must be verified on unpowered attach. JP1 OPEN = OFF (default). Close RUN ONLY for an approved dedicated source. PG is diagnostic, not a current-cont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"
- note added: "STOP: NO INPUT TVS / ESD OR SURGE PROTECTION - DO NOT FABRICATE"
- note removed: "9 V request only. No USB data. CH224K Rd must be verified on unpowered attach. JP1 OPEN = OFF (default). Close ONLY for an approved dedicated source. PG is diagnostic, not a current-contract detector. No series diode: TPS26600 reverse-current blocking is specified; qualify dead-battery/backfeed on hardware. All bulk capacitance is behind the eFuse. No legacy-host enumeration or CC-current decodin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"
Changed lines of the file:
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@@
 (kicad_sch (version 20250114) (generator "eeschema") (paper "A3") (title_block (title "USB-C sink / permission / protected input") (date "2026-09-24") (rev "A0 ENGINEERING PROTOTYPE") (company "Big Modular") (comment 1 "NOT FOR FABRICATION - UNROUTED PLACEMENT SCAFFOLDS"))
 (text "USB-C sink / permission / protected input" (at 16 15 0) (effects (font (size 2 2)) (justify left)))
-(text "9 V request only. No USB data. CH224K Rd must be verified on unpowered attach.\nJP1 OPEN = OFF (default). Close ONLY for an approved dedicated source. PG is diagnostic, not a current-contract detector.\nNo series diode: TPS26600 reverse-current blocking is specified; qualify dead-battery/backfeed on hardware.\nAll bulk capacitance is behind the eFuse. No legacy-host enumeration or CC-current decoding is implemented." (at 16 27 0) (effects (font (size 1.05 1.05)) (justify left)))
+(text "STOP: NO INPUT TVS / ESD OR SURGE PROTECTION - DO NOT FABRICATE" (at 16 25 0) (effects (font (size 1.9 1.9)) (justify left)))
+(text "D1 SMBJ12CA REMOVED: it can burn at sustained 15/20 V. F1 (500 mA / 32 V) is NOT a coordinated surge fuse.\nTPS26600 OVP (~10.8 V) disconnects OUTPUT, not upstream VBUS. No qualified VBUS transient protection.\n9 V request only. No USB data. CH224K Rd must be verified on unpowered attach. JP1 OPEN = OFF (default).\nClose RUN ONLY for an approved dedicated source. PG is diagnostic, not a current-contract detector.\nNo series diode: TPS26600 reverse-current blocking is specified; qualify dead-battery/backfeed on hardware.\nAll bulk capacitance is behind the eFuse. No legacy-host enumeration or CC-current decoding is implemented." (at 16 34 0) (effects (font (size 1.05 1.05)) (justify left)))
 (wire (pts (xy 41.91 87.63) (xy 41.91 92.71)) (stroke (width 0) (type default)))
 (global_label "GND" (shape bidirectional) (at 41.91 92.71 270) (effects (font (size 0.85 0.85))))
@@
 (wire (pts (xy 41.91 133.35) (xy 41.91 138.43)) (stroke (width 0) (type default)))
 (global_label "VBUS_FUSED" (shape bidirectional) (at 41.91 138.43 270) (effects (font (size 0.85 0.85))))
-(symbol (lib_id "BigModular:Device_Fuse") (at 41.91 129.54 0) (unit 1) (in_bom yes) (on_board yes) (dnp no)(property "Reference" "F1" (at 41.91 120.64999999999999 0) (effects (font (size 1.15 1.15))))(property "Value" "500mA 32V fuse" (at 41.91 123.19 0) (effects (font (size 1.05 1.05))))(property "Footprint" "" (at 41.91 129.54 0) (effects (font (size 1 1)) hide))(property "MPN" "" (at 41.91 129.54 0) (effects (font (size 1 1)) hide))(property "LCSC" "" (at 41.91 129.54 0) (effects (font (size 1 1)) hide))(property "NOTE" "Candidate rating, NOT USB current authorization or coordinated surge qualification." (at 41.91 129.54 0) (effects (font (size 1 1)) hide))(pin "1")(pin "2")(instances (project "big_modular" (path "/d567704c-57ad-5df1-b183-cadb01fd8972/029cb2a9-d2ef-5d6a-923b-0d0afe15605f" (reference "F1") (unit 1)))) )
-(wire (pts (xy 120.64999999999999 129.54) (xy 115.57 129.54)) (stroke (width 0) (type default)))
-(global_label "VBUS_FUSED" (shape bidirectional) (at 115.57 129.54 180) (effects (font (size 0.85 0.85))))
-(wire (pts (xy 128.26999999999998 129.54) (xy 133.35 129.54)) (stroke (width 0) (type default)))
-(global_label "GND" (shape bidirectional) (at 133.35 129.54 0) (effects (font (size 0.85 0.85))))
-(symbol (lib_id "BigModular:Device_D_TVS") (at 124.46 129.54 0) (unit 1) (in_bom yes) (on_board yes) (dnp no)(property "Reference" "D1" (at 124.46 124.46 0) (effects (font (size 1.15 1.15))))(property "Value" "SMBJ12CA" (at 124.46 127.0 0) (effects (font (size 1.05 1.05))))(property "Footprint" "" (at 124.46 129.54 0) (effects (font (size 1 1)) hide))(property "MPN" "SMBJ12CA" (at 124.46 129.54 0) (effects (font (size 1 1)) hide))(property "LCSC" "" (at 124.46 129.54 0) (effects (font (size 1 1)) hide))(property "NOTE" "12V standoff: sustained 15/20V is a TVS/fuse fault, NOT qualified OV protection." (at 124.46 129.54 0) (effects (font (size 1 1)) hide))(pin "1")(pin "2")(instances (project "big_modular" (path "/d567704c-57ad-5df1-b183-cadb01fd8972/029cb2a9-d2ef-5d6a-923b-0d0afe15605f" (reference "D1") (unit 1)))) )
+(symbol (lib_id "BigModular:Device_Fuse") (at 41.91 129.54 0) (unit 1) (in_bom yes) (on_board yes) (dnp no)(property "Reference" "F1" (at 41.91 120.64999999999999 0) (effects (font (size 1.15 1.15))))(property "Value" "500mA 32V fuse" (at 41.91 123.19 0) (effects (font (size 1.05 1.05))))(property "Footprint" "" (at 41.91 129.54 0) (effects (font (size 1 1)) hide))(property "MPN" "" (at 41.91 129.54 0) (effects (font (size 1 1)) hide))(property "LCSC" "" (at 41.91 129.54 0) (effects (font (size 1 1)) hide))(property "NOTE" "Unselected candidate: 32V rating covers steady 20/21V only; interrupt/surge ratings, time-current and source coordination UNQUALIFIED. Not USB current authorization." (at 41.91 129.54 0) (effects (font (size 1 1)) hide))(pin "1")(pin "2")(instances (project "big_modular" (path "/d567704c-57ad-5df1-b183-cadb01fd8972/029cb2a9-d2ef-5d6a-923b-0d0afe15605f" (reference "F1") (unit 1)))) )
 (wire (pts (xy 270.51 125.72999999999999) (xy 270.51 120.65)) (stroke (width 0) (type default)))
 (global_label "VBUS_FUSED" (shape bidirectional) (at 270.51 120.65 90) (effects (font (size 0.85 0.85))))
 (wire (pts (xy 270.51 133.35) (xy 270.51 138.43)) (stroke (width 0) (type default)))
 (global_label "GND" (shape bidirectional) (at 270.51 138.43 270) (effects (font (size 0.85 0.85))))
-(symbol (lib_id "BigModular:Device_C") (at 270.51 129.54 0) (unit 1) (in_bom yes) (on_board yes) (dnp no)(property "Reference" "C2" (at 270.51 120.64999999999999 0) (effects (font (size 1.15 1.15))))(property "Value" "100n 50V" (at 270.51 123.19 0) (effects (font (size 1.05 1.05))))(property "Footprint" "Capacitor_SMD:C_1206_3216Metric" (at 270.51 129.54 0) (effects (font (size 1 1)) hide))(property "MPN" "" (at 270.51 129.54 0) (effects (font (size 1 1)) hide))(property "LCSC" "" (at 270.51 129.54 0) (effects (font (size 1 1)) hide))(property "NOTE" "" (at 270.51 129.54 0) (effects (font (size 1 1)) hide))(pin "1")(pin "2")(instances (project "big_modular" (path "/d567704c-57ad-5df1-b183-cadb01fd8972/029cb2a9-d2ef-5d6a-923b-0d0afe15605f" (reference "C2") (unit 1)))) )
+(symbol (lib_id "BigModular:Device_C") (at 270.51 129.54 0) (unit 1) (in_bom yes) (on_board yes) (dnp no)(property "Reference" "C2" (at 270.51 120.64999999999999 0) (effects (font (size 1.15 1.15))))(property "Value" "100n 50V" (at 270.51 123.19 0) (effects (font (size 1.05 1.05))))(property "Footprint" "Capacitor_SMD:C_1206_3216Metric" (at 270.51 129.54 0) (effects (font (size 1 1)) hide))(property "MPN" "" (at 270.51 129.54 0) (effects (font (size 1 1)) hide))(property "LCSC" "" (at 270.51 129.54 0) (effects (font (size 1 1)) hide))(property "NOTE" "TPS26600 local bypass only. Not an ESD/surge clamp; effective capacitance and hot-plug transients unverified." (at 270.51 129.54 0) (effects (font (size 1 1)) hide))(pin "1")(pin "2")(instances (project "big_modular" (path "/d567704c-57ad-5df1-b183-cadb01fd8972/029cb2a9-d2ef-5d6a-923b-0d0afe15605f" (reference "C2") (unit 1)))) )
 (no_connect (at 59.69 204.47))
 (no_connect (at 80.00999999999999 213.36))
