File: hardware/06_sensing.kicad_sch (KiCad schematic)
At the start: 40 parts, among them U11 TLV9002IDR

Commit message: Clarify hierarchical ports and replace local label islands with visible schematic wiring
Other:
- moved on the sheet: C41, R43
