File: hardware/big_modular.kicad_sch (KiCad schematic)
At the start: 88 parts, among them J1 USB4105-GF-A, J2 16-pin IDC POWER OUT, Q1 MMBT3906, U1 CH224K, U2 TPS26600PWPR, U3 TPS62160DSGR, U4 TPS65131RGER, U5 TPS62125DSGR, U6 TPS7A4901DGNR, U7 TPS7A3001DGNR, U8 TPS7A4901DGNR

Commit message: Simple schematics.
Parts:
- removed C1: 1u 50V X7R, Capacitor_SMD:C_1206_3216Metric, symbol BigModular:Device_C
- removed C10, C11: 6.8p C0G 50V, Capacitor_SMD:C_1206_3216Metric, symbol BigModular:Device_C
- removed C12: 220n 10V, Capacitor_SMD:C_1206_3216Metric, symbol BigModular:Device_C
- removed C13, C23, C24, C27, C28, C31, C32: 10n 50V, Capacitor_SMD:C_1206_3216Metric, symbol BigModular:Device_C
- removed C14: 4.7n C0G 50V, Capacitor_SMD:C_1206_3216Metric, symbol BigModular:Device_C
- removed C15: 100n 10V, Capacitor_SMD:C_1206_3216Metric, symbol BigModular:Device_C
- removed C16, C17: 4.7u 10V X7R, Capacitor_SMD:C_1206_3216Metric, symbol BigModular:Device_C
- removed C18, C21, C22, C25, C26, C29, C30, C4, C5: 10u 25V X7R, Capacitor_SMD:C_1206_3216Metric, symbol BigModular:Device_C
- removed C19: 22u 16V X7R, Capacitor_SMD:C_1206_3216Metric, symbol BigModular:Device_C
- removed C2, C3: 100n 50V, Capacitor_SMD:C_1206_3216Metric, symbol BigModular:Device_C
- removed C20, C7: 100n 25V, Capacitor_SMD:C_1206_3216Metric, symbol BigModular:Device_C
- removed C6: 22u 10V X7R, Capacitor_SMD:C_1206_3216Metric, symbol BigModular:Device_C
- removed C8, C9: 22u 25V X7R, Capacitor_SMD:C_1206_3216Metric, symbol BigModular:Device_C
- removed D2, D3, D4, D5, D6, D7, D8, D9: Schottky 1A 40V, symbol BigModular:Device_D_Schottky
- removed F1: 500mA 32V fuse, symbol BigModular:Device_Fuse
- removed J1: USB4105-GF-A, BigModular:USB_C_Receptacle_GCT_USB4105-xx-A_16P_TopMnt_Horizontal, symbol BigModular:Connector_USB_C_Receptacle_USB2.0_16P
- removed J2: 16-pin IDC POWER OUT, symbol BigModular:Connector_Generic_Conn_02x08_Odd_Even
- removed JP1: RUN / default OPEN, symbol BigModular:Jumper_Jumper_2_Open
- removed L1: 2.2uH / Isat>=2A, symbol BigModular:Device_L
- removed L2, L3: 4.7uH / Isat>=3A, symbol BigModular:Device_L
- removed L4: 10uH / Isat>=1A, symbol BigModular:Device_L
- removed Q1: MMBT3906, Package_TO_SOT_SMD:SOT-23, symbol BigModular:Transistor_BJT_MMBT3906
- removed R1: 1k 1% >=0.5W, Resistor_SMD:R_2010_5025Metric, symbol BigModular:Device_R
- removed R10, R18, R20, R22, R24: 10k 0.1%, Resistor_SMD:R_0603_1608Metric, symbol BigModular:Device_R
- removed R11, R25, R26, R3: 100k, Resistor_SMD:R_0603_1608Metric, symbol BigModular:Device_R
- removed R12: 1.05M 0.1%, Resistor_SMD:R_0603_1608Metric, symbol BigModular:Device_R
- removed R13, R15: 100k 0.1%, Resistor_SMD:R_0603_1608Metric, symbol BigModular:Device_R
- removed R14: 1.15M 0.1%, Resistor_SMD:R_0603_1608Metric, symbol BigModular:Device_R
- removed R16: 100R, Resistor_SMD:R_0603_1608Metric, symbol BigModular:Device_R
- removed R17: 71.5k 0.1%, Resistor_SMD:R_0603_1608Metric, symbol BigModular:Device_R
- removed R19: 91.2k 0.1%, Resistor_SMD:R_0603_1608Metric, symbol BigModular:Device_R
- removed R2: 6.8k 1%, Resistor_SMD:R_0603_1608Metric, symbol BigModular:Device_R
- removed R21: 92k 0.1%, Resistor_SMD:R_0603_1608Metric, symbol BigModular:Device_R
- removed R23: 32.2k 0.1%, Resistor_SMD:R_0603_1608Metric, symbol BigModular:Device_R
- removed R27: 47k, Resistor_SMD:R_0603_1608Metric, symbol BigModular:Device_R
- removed R28: 22k 1%, Resistor_SMD:R_0603_1608Metric, symbol BigModular:Device_R
- removed R29, R5, R7: 100k 1%, Resistor_SMD:R_0603_1608Metric, symbol BigModular:Device_R
- removed R30, R31: 10k 1%, Resistor_SMD:R_0603_1608Metric, symbol BigModular:Device_R
- removed R4: 562k 1%, Resistor_SMD:R_0603_1608Metric, symbol BigModular:Device_R
- removed R6: 806k 1%, Resistor_SMD:R_0603_1608Metric, symbol BigModular:Device_R
- removed R8: 40.2k 1%, Resistor_SMD:R_0603_1608Metric, symbol BigModular:Device_R
- removed R9: 40.2k 0.1%, Resistor_SMD:R_0603_1608Metric, symbol BigModular:Device_R
- removed U1: CH224K, Package_SO:SSOP-10-1EP_3.9x4.9mm_P1mm_EP2.1x3.3mm, symbol BigModular:Interface_USB_CH224K
- removed U2: TPS26600PWPR, Package_SO:HTSSOP-16-1EP_4.4x5mm_P0.65mm_EP3.4x5mm_Mask2.66x2.46mm_ThermalVias, symbol BigModular:Power_Management_TPS26600PWP
- removed U3: TPS62160DSGR, Package_SON:Texas_DSG0008A_WSON-8-1EP_2x2mm_P0.5mm_EP0.9x1.6mm_ThermalVias, symbol BigModular:Regulator_Switching_TPS62160DSG
- removed U4: TPS65131RGER, Package_DFN_QFN:VQFN-24-1EP_4x4mm_P0.5mm_EP2.45x2.45mm_ThermalVias, symbol BigModular:Regulator_Switching_TPS65131RGE
- removed U5: TPS62125DSGR, symbol BigModular:TPS62125DSGR
- removed U6, U8: TPS7A4901DGNR, symbol BigModular:TPS7A4901DGNR
- removed U7: TPS7A3001DGNR, symbol BigModular:TPS7A3001DGNR
Connections:
- no-connect marks 28 -> 0
Other:
- added sheet Input and protection (01_input_protection.kicad_sch)
- added sheet Output rails (03_output_rails.kicad_sch)
- added sheet Power conversion (02_power_conversion.kicad_sch)
- note added: "BIG MODULAR / SCHEMATIC MAP"
- note added: "HOW TO READ Open each sheet in KiCad or click its box in the PDF. Local feedback, filtering and protection networks use real wires. Named ports carry power between sheets; GND is shared, RTN is not."
- note added: "INCOMPLETE / NON-OPERATIONAL / DO NOT FABRICATE"
- note added: "LIMITS: No PDO/current proof, qualified input surge protection or completed PCB layout. Read docs/schematic-guide.md and docs/component-guide.md."
- note added: "Three LDOs / J2 See page 4"
- note added: "Three functional subsheets | 88 real components | Circuit connectivity retained"
- note added: "USB-C / CH224K Fuse + eFuse PG / RUN / voltage gate See page 2"
- note added: "V4 intermediate Bipolar boost / inverter +5 V preregulation See page 3"
- note removed: "+12 V POSTREG"
- note removed: "+5 V POSTREG"
- note removed: "-12 V POSTREG"
- note removed: "4.016 V BUCK"
- note removed: "5 V VBUS powers negotiation only. Gate = PG active LOW AND 7.88..10.78 V nominal window AND RUN. NO 5 V OUTPUT MODE."
- note removed: "6.52 V BUCK"
- note removed: "9 V REQUEST / PG INTERLOCK"
- note removed: "9 V must be independently verified by PD analyzer at >=0.5 A contract before any test. About 40 mA/rail simultaneous TEST LOADS ONLY; no rating."
- note removed: "BIG MODULAR | PD-ONLY 9 V | ONE CONNECTED CIRCUIT | A1 WIP"
- note removed: "BIPOLAR +/-13.95 V"
- note removed: "BLOCKERS: PG does NOT prove PDO/current. No qualified input ESD/surge protection. J1 has four physical DRC violations."
- note removed: "No TVS fitted: D1 reference reserved. Do not substitute a 12 V-standoff clamp on upstream USB VBUS. LDOs are not precision output-OVP devices. No all-rail shutdown/tracking or rapid discharge guarantee. Read docs/design-review.md, mechanics.md and reports/validation-summary.md. Converter stability, thermals, surge and physical fit remain untested."
- note removed: "OFF-BOARD J2"
- note removed: "POWER/RETURN DECLARATIONS (not PCB pads)"
- note removed: "R4/R5: 562k/100k UV; R6/R7: 806k/100k OV. SHDN LOW = OFF. JP1 cannot override either window limit. PG generic active-low OD, not authenticated contract/current. Default RUN OPEN. RTN is NOT externally shorted to GND."
- note removed: "STOP: PCB has only J1 and mechanical holes. No tracks / vias / zones. Neither board is operational."
- note removed: "U4 PSP/PSN grounded; BSW intentionally unused. Positive boost can prebias only AFTER the gated V4 supply exists. Negative feedback lower resistor returns to BI_REF, not GND. PG of U3 holds both U4 enables low during intermediate startup."
- note removed: "USB-C / FUSE"
- note removed: "eFUSE / UV + OV"
- title: Big Modular - PD ONLY / one-sheet circuit proposal -> Big Modular - Overview and sheet navigation

Commit message: Save 9 V power-supply schematic prototype and LED mechanical provisions
Other:
- sheet Input and protection renamed USB PD and always-on housekeeping
- removed sheet Output rails
- removed sheet Power conversion
- added sheet Always-on MCU and indicators (05_diagnostics.kicad_sch)
- added sheet Direct bipolar rails (04_bipolar.kicad_sch)
- added sheet Independent buck converters (03_bucks.kicad_sch)
- added sheet Independent hardware gate (02_hardgate.kicad_sch)
- added sheet Manual output harness (07_output_rails.kicad_sch)
- added sheet Rail sensing and input protection (06_sensing.kicad_sch)
- sheet USB PD and always-on housekeeping ports: added AUX3V3, PD_PG_N, PD_SCL, PD_SDA, VBUS_FUSED, VBUS_RAW; removed VPROT
- note added: "BIG MODULAR / 9 V PD ELECTRICAL PROTOTYPE"
- note added: "CONNECTED REVIEW CANDIDATE - NOT QUALIFIED FOR POWER-UP OR FABRICATION"
- note added: "READ docs/electrical-prototype.md + firmware/README.md. RUN OPEN; firmware default DENY. Main stages: TPS54302 MID -> TPS65131 direct +/-12 V; separate TPS54302 +5 V. Mechanics retained; PCB NOT synchronized or routed. Native parity intentionally incomplete."
- note removed: "BIG MODULAR / SCHEMATIC MAP"
- note removed: "HOW TO READ Open each sheet in KiCad or click its box in the PDF. Local feedback, filtering and protection networks use real wires. Named ports carry power between sheets; GND is shared, RTN is not."
- note removed: "INCOMPLETE / NON-OPERATIONAL / DO NOT FABRICATE"
- note removed: "LIMITS: No PDO/current proof, qualified input surge protection or completed PCB layout. Read docs/schematic-guide.md and docs/component-guide.md."
- note removed: "Three LDOs / J2 See page 4"
- note removed: "Three functional subsheets | 88 real components | Circuit connectivity retained"
- note removed: "USB-C / CH224K Fuse + eFuse PG / RUN / voltage gate See page 2"
- note removed: "V4 intermediate Bipolar boost / inverter +5 V preregulation See page 3"
- title: Big Modular - Overview and sheet navigation -> Big Modular - Electrical prototype / hierarchy

Commit message: Replace MCU diagnostics with optional rail-sense IDC and single 5 V power LED
Other:
- sheet Always-on MCU and indicators renamed Rail debug and single power LED
- sheet Direct bipolar rails ports: added none; removed BI_EN
- sheet Independent hardware gate ports: added none; removed MCU_PERMIT_N
- sheet Rail debug and single power LED ports: added P5; removed BI_EN, MCU_PERMIT_N
- note added: "READ docs/electrical-prototype.md + docs/debug-interface.md. RUN OPEN for qualification; hardware-only operation, no debug MCU. Main stages: TPS54302 MID -> TPS65131 direct +/-12 V; separate TPS54302 +5 V. Mechanics retained; PCB NOT synchronized or routed. Native parity intentionally incomplete."
- note removed: "READ docs/electrical-prototype.md + firmware/README.md. RUN OPEN; firmware default DENY. Main stages: TPS54302 MID -> TPS65131 direct +/-12 V; separate TPS54302 +5 V. Mechanics retained; PCB NOT synchronized or routed. Native parity intentionally incomplete."

Commit message: Clarify hierarchical ports and replace local label islands with visible schematic wiring
Other:
- note added: "6 protected channels"
- note added: "BIG MODULAR / WIRED POWER FLOW"
- note added: "J7 -> cable -> J2"
- note added: "J7 PCB landing -> one flying lead -> J2 keyed POWER OUT Flag-only ports at bottom preserve independent ERC declarations. RTN stays local to hardware gate; never substitute GND."
- note added: "J8 DEBUG / D10 LED"
- note added: "REVIEW ONLY - NOT QUALIFIED FOR POWER-UP OR FABRICATION"
- note added: "SENSE -> DEBUG: six protected analog outputs J8 optional20-pin DEBUG ONLY; NOT POWER. No MCU, blink or external enable dependency."
- note added: "U2 / UV-OV + PG"
- note added: "U3 MID / U5 +5V"
- note added: "U4 / +/-12V"
- note added: "USB-C / PD + AUX"
- note removed: "BIG MODULAR / 9 V PD ELECTRICAL PROTOTYPE"
- note removed: "CONNECTED REVIEW CANDIDATE - NOT QUALIFIED FOR POWER-UP OR FABRICATION"
- note removed: "READ docs/electrical-prototype.md + docs/debug-interface.md. RUN OPEN for qualification; hardware-only operation, no debug MCU. Main stages: TPS54302 MID -> TPS65131 direct +/-12 V; separate TPS54302 +5 V. Mechanics retained; PCB NOT synchronized or routed. Native parity intentionally incomplete."

Commit message: Simplify V1 power architecture, remove auxiliary sensing and obsolete documentation, enable autonomous protected start and reset button
Other:
- sheet Independent hardware gate renamed Autonomous hardware window and retry
- sheet Manual output harness renamed Board output and power LED
- sheet USB PD and always-on housekeeping renamed USB PD input
- removed sheet Rail debug and single power LED
- removed sheet Rail sensing and input protection
- sheet Autonomous hardware window and retry ports: added VIN9; removed AUX3V3, EF_ENABLE, EF_FLT_N, PD_PG_N, VBUS_FUSED
- sheet Board output and power LED ports: added none; removed ANA_MID, MID, VBUS_FUSED, VBUS_RAW
- sheet Direct bipolar rails ports: added none; removed ANA_MID
- sheet Independent buck converters ports: added none; removed EF_ENABLE
- sheet USB PD input ports: added VIN9; removed AUX3V3, PD_PG_N, PD_SCL, PD_SDA, VBUS_FUSED, VBUS_RAW
- note added: "9 V voltage acceptance is NOT proof of a PD protocol contract. No MCU, AUX regulator, sensing/debug or artificial RUN inhibit. SW1 retries eFuse; UV/OV window remains independent."
- note added: "AUTONOMOUS 9 V INPUT / UNROUTED / NOT A MANUFACTURING RELEASE"
- note added: "J7 / D10 P5 LED"
- note added: "J7 is the physical output boundary; one manual harness. USB/button/LED will move together near panel top in later mechanics. PCB placement and all copper are untouched by this revision."
- note added: "U2 WINDOW / SW1 RETRY"
- note added: "USB-C / FIXED9V"
- note removed: "6 protected channels"
- note removed: "J7 -> cable -> J2"
- note removed: "J7 PCB landing -> one flying lead -> J2 keyed POWER OUT Flag-only ports at bottom preserve independent ERC declarations. RTN stays local to hardware gate; never substitute GND."
- note removed: "J8 DEBUG / D10 LED"
- note removed: "REVIEW ONLY - NOT QUALIFIED FOR POWER-UP OR FABRICATION"
- note removed: "SENSE -> DEBUG: six protected analog outputs J8 optional20-pin DEBUG ONLY; NOT POWER. No MCU, blink or external enable dependency."
- note removed: "U2 / UV-OV + PG"
- note removed: "USB-C / PD + AUX"
- title: Big Modular - Electrical prototype / hierarchy -> Big Modular - V1 electrical hierarchy
