File: hardware/big_modular.kicad_pcb (KiCad board)
At the start: 4 copper layers, 100.5 x 30 mm, 68 parts, among them J1 TYPE-C-31-M-12, J7 Manual IDC wire landing, SW1 TL3340AF160QG, U1 CH224A, U2 TPS26600PWPR, U3 TPS54302DDCR, U4 TPS65131RGER, U5 TPS54302DDCR

Commit message: Add low-noise ±12 V LDO prototype supply and verified LDO-R1 fabrication release
Parts:
- added C48: 22u 25V X5R, BigModular:C_1206_3216Metric, F.Cu at (109.2, 81.7)
- added C49: 22u 25V X5R, BigModular:C_1206_3216Metric, F.Cu at (109.6, 86.6)
- added C50: 22u 25V X5R, BigModular:C_1206_3216Metric, F.Cu at (113.3, 86.1)
- added C51: 22u 25V X5R, BigModular:C_1206_3216Metric, F.Cu at (98.8, 81.0)
- added C52: 22u 25V X5R, BigModular:C_1206_3216Metric, F.Cu at (98.8, 83.6)
- added C53: 22u 25V X5R, BigModular:C_1206_3216Metric, F.Cu at (98.8, 86.2)
- added C54: 22u 25V X5R, BigModular:C_1206_3216Metric, F.Cu at (65.0, 74.5)
- added C55: 22u 25V X5R, BigModular:C_1206_3216Metric, F.Cu at (65.0, 77.1)
- added C56: 22u 25V X5R, BigModular:C_1206_3216Metric, F.Cu at (65.0, 79.7)
- added C57: 22u 25V X5R, BigModular:C_1206_3216Metric, F.Cu at (52.7, 74.5)
- added C58: 22u 25V X5R, BigModular:C_1206_3216Metric, F.Cu at (52.7, 77.1)
- added C59: 22u 25V X5R, BigModular:C_1206_3216Metric, F.Cu at (52.7, 79.7)
- added C60: 1u 50V X7R, BigModular:C_0805_2012Metric, F.Cu at (108.5, 90.5)
- added C61: 100n 50V X7R, BigModular:C_0603_1608Metric, F.Cu at (64.5, 82.6)
- added C62: 10n 50V X7R, BigModular:C_0603_1608Metric, F.Cu at (55.5, 83.9)
- added C63: 22u 25V X5R, BigModular:C_1206_3216Metric, B.Cu at (113.3, 86.1)
- added C64: 22u 25V X5R, BigModular:C_1206_3216Metric, B.Cu at (98.8, 81.0)
- added C65: 22u 25V X5R, BigModular:C_1206_3216Metric, B.Cu at (98.8, 83.6)
- added C66: 22u 25V X5R, BigModular:C_1206_3216Metric, B.Cu at (98.8, 87.9)
- added C67: 22u 25V X5R, BigModular:C_1206_3216Metric, F.Cu at (68.8, 82.6)
- added D27: SS34 40V, BigModular:D_SMA, F.Cu at (104.8, 87.6)
- added D28: SS34 40V, BigModular:D_SMA, F.Cu at (71.0, 76.3)
- added R72: 90.9k 0.1%, BigModular:R_0603_1608Metric, F.Cu at (52.5, 82.5)
- added R73: 1.21k 0.1%, BigModular:R_0603_1608Metric, F.Cu at (55.5, 82.3)
- added R74: 10k 0.1%, BigModular:R_0603_1608Metric, F.Cu at (58.5, 83.0)
- added R75: 23.2k 0.1%, BigModular:R_0603_1608Metric, F.Cu at (125.6, 73.8)
- added R76: 2.49k 0.1%, BigModular:R_0603_1608Metric, F.Cu at (134.8, 79.0)
- added U12: TPS7A4700RGWR, BigModular:Texas_RGW0020A_VQFN-20-1EP_5x5mm_P0.65mm_EP3.15x3.15mm, F.Cu at (104.5, 82.6)
- added U13: TPS7A3301RGWR, BigModular:Texas_RGW0020A_VQFN-20-1EP_5x5mm_P0.65mm_EP3.15x3.15mm, F.Cu at (59.0, 77.7)
- C10: value 6.8p 50V C0G -> 4.5p 50V C0G
- C11: value 6.8p 50V C0G -> 4.3p 50V C0G
- R12: value 1.33M 1% -> 1.5M 0.1%; footprint BigModular:R_0603_1608Metric -> BigModular:R_0805_2012Metric
- R13, R15, R60: value 150k 1% -> 150k 0.1%
- R14: value 1.33M 1% -> 1.6M 0.1%; footprint BigModular:R_0603_1608Metric -> BigModular:R_0805_2012Metric
- moved R26 68.9 mm to (70.8, 80.0), turned to 180 degrees
- moved C37 25.5 mm to (139.4, 81.5)
- moved R25 12.2 mm to (98.8, 88.5), turned to 180 degrees
- moved R27 1.50 mm to (94.9, 84.5)
- moved R12 0.25 mm to (122.2, 75.2)
Connections:
- C10 pad 1: /P12 -> /Direct bipolar rails/PRAW
- C11 pad 1: /N12 -> /Direct bipolar rails/NRAW
- C8 pad 1: /P12 -> /Direct bipolar rails/PRAW
- C9 pad 1: /N12 -> /Direct bipolar rails/NRAW
- D2 pad 1: /P12 -> /Direct bipolar rails/PRAW
- D3 pad 2: /N12 -> /Direct bipolar rails/NRAW
- R12 pad 1: /P12 -> /Direct bipolar rails/PRAW
- R12 pad 2: /Direct bipolar rails/POS_FB -> /Direct bipolar rails/POS_DIV
- R14 pad 1: /N12 -> /Direct bipolar rails/NRAW
- R15 pad 2: /Direct bipolar rails/BI_REF -> /Direct bipolar rails/NEG_REF_DIV
- U4 pad 15: /N12 -> /Direct bipolar rails/NRAW
- U4 pad 23: /P12 -> /Direct bipolar rails/PRAW
Routing:
- net /Direct bipolar rails/NRAW: track 0.00 -> 177.5 mm, vias 0 -> 9
- net /Direct bipolar rails/PRAW: track 0.00 -> 68.3 mm, vias 0 -> 8
- net /N12: track 129.4 -> 64.1 mm, vias 7 -> 5
- net /MID: track 91.1 -> 116.2 mm, vias 8 -> 11
- net /Quiet bipolar post-regulators/N_LDO_FB: track 0.00 -> 12.3 mm, vias 0 -> 2
- net /Quiet bipolar post-regulators/P_NR: track 0.00 -> 9.52 mm, vias 0 -> 2
- net /Quiet bipolar post-regulators/N_LDO_DIV: track 0.00 -> 9.40 mm
- net /GND: track 79.8 -> 88.2 mm, vias 49 -> 90
- net /P12: track 59.9 -> 51.6 mm, vias 6 -> 2
- net /Quiet bipolar post-regulators/N_NR: track 0.00 -> 7.46 mm, vias 0 -> 2
- net /P5: track 84.8 -> 81.7 mm, vias 10 -> 8
- net /Direct bipolar rails/BI_REF: track 9.01 -> 11.9 mm, vias 0 -> 2
- net /Direct bipolar rails/POS_DIV: track 0.00 -> 2.25 mm
- net /VPROT: track 92.4 -> 90.9 mm
- net /Direct bipolar rails/NEG_REF_DIV: track 0.00 -> 1.48 mm
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- added copper zone on B.Cu, net /GND
- added copper zone on F.Cu, net /GND
