File: hardware/05_quiet_rails.kicad_sch (KiCad schematic)
At the start: 27 parts, among them U12 TPS7A4700RGWR, U13 TPS7A3301RGWR

Commit message: Apply Basic passive substitutions with corrected dividers, 1206 capacitor routing and verified prototype release
Parts:
- added R83: 9.1k 1%, BigModular:R_0603_1608Metric, symbol BigModular:Device_R
- R72: value 90.9k 0.1% -> 82k 1%; LCSC C728600 -> C23254; MPN RT0603BRD0790K9L -> 0603WAF8202T5E; Manufacturer YAGEO -> UNI-ROYAL(Uniroyal Elec); NOTE Precision negative divider: (90.9k+1.21k)/10k; -11.997925V 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 -> Basic negative divider:(82k+9.1k+1.2k)/10k=-12.02025V befor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
- R73: value 1.21k 0.1% -> 1.2k 1%; LCSC C705737 -> C22765; MPN RT0603BRD071K21L -> 0603WAF1201T5E; Manufacturer YAGEO -> UNI-ROYAL(Uniroyal Elec); NOTE Precision negative divider: (90.9k+1.21k)/10k; -11.997925V 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 -> Basic negative divider:(82k+9.1k+1.2k)/10k=-12.02025V befor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
- R74: value 10k 0.1% -> 10k 1%; LCSC C95204 -> C25804; MPN RT0603BRD0710KL -> 0603WAF1002T5E; Manufacturer YAGEO -> UNI-ROYAL(Uniroyal Elec); NOTE Precision negative divider: (90.9k+1.21k)/10k; -11.997925V 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 -> Basic negative divider:(82k+9.1k+1.2k)/10k=-12.02025V befor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
Connections:
- net N_LDO_DIV: now also R83.2; no longer R72.2
- new net N_LDO_SER: R72.2, R83.1
Other:
- note added: "(R72+R83+R73)/R74 =92.3k/10k -> -12.02025V before IFB; 117.5uA nominal divider current (>5uA required). C61 100n: typical ~120ms start, not rail sequencing. C62 10n improves AC; shutdown FB kick remains a test gate. D27/D28 divert reverse current, do NOT block it. SS34 Vf does NOT prove the negative -0.3V differential limit. 800mA aspiration is load-dependent, not a simultaneous rail guarantee. C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"
- note added: "Raw +13.537080/-13.928806V remain internal. Final +5V is unchanged and bypasses this sheet. Both exposed pads 21 are GND. Exact requested RGWR parts; NOT a +/-1A supply."
- note removed: "R72+R73 / R74 = 92.11k / 10k -> -11.997925V before IFB; 117.5uA nominal divider current (>5uA required). C61 100n: typical ~120ms start, not rail sequencing. C62 10n improves AC; shutdown FB kick remains a test gate. D27/D28 divert reverse current, do NOT block it. SS34 Vf does NOT prove the negative -0.3V differential limit. 800mA aspiration is load-dependent, not a simultaneous rail guarantee. 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"
- note removed: "Raw +13.530611/-13.920585V remain internal. Final +5V is unchanged and bypasses this sheet. Both exposed pads 21 are GND. Exact requested RGWR parts; NOT a +/-1A supply."
