File: modules/usb-power/hardware/05_quiet_rails.kicad_sch (KiCad schematic)
At the start: 28 parts, among them U12 TPS7A4700RGWR, U13 TPS7A3301RGWR

Commit message: Save exact Astra SR2 schematic candidate and DeepSeek review; keep PCB unchanged
Parts:
- added C73, C74: 22u 25V X5R, BigModular:C_1206_3216Metric, symbol BigModular:Device_C
- C54, C55, C56, C67: NOTE negative input bank: 4 parallel CL31A226KAHNNNE. Prototype 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 -> negative input bank: 5 parallel CL31A226KAHNNNE. Prototype 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
- C57, C58, C59: NOTE negative output bank: 3 parallel CL31A226KAHNNNE. Prototype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 -> negative output bank: 4 parallel CL31A226KAHNNNE. Prototype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
- C62: JLCPCB Audit Requirements (none) -> {"reason": "C62 prototype DNP: retain pads, noise/PSRR trad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; JLCPCB Exclude (none) -> yes; NOTE 10n from OUT to FB across entire upper divider. Improves AC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 -> DNP prototype: retain pads; TI TPS7A33 section8.1.4 says CF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; now not fitted
- R72: value 82k 1% -> 90.9k 0.1%; LCSC C23254 -> C728600; MPN 0603WAF8202T5E -> RT0603BRD0790K9L; Manufacturer UNI-ROYAL(Uniroyal Elec) -> YAGEO; NOTE Basic negative divider:(82k+9.1k+1.2k)/10k=-12.02025V befor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 -> SR1 final divider:(90.9k+0R+1.2k)/10k=-11.99675V before IFB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
- R73: NOTE Basic negative divider:(82k+9.1k+1.2k)/10k=-12.02025V befor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 -> SR1 final divider:(90.9k+0R+1.2k)/10k=-11.99675V before IFB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
- R74: value 10k 1% -> 10k 0.1%; LCSC C25804 -> C95204; MPN 0603WAF1002T5E -> RT0603BRD0710KL; Manufacturer UNI-ROYAL(Uniroyal Elec) -> YAGEO; NOTE Basic negative divider:(82k+9.1k+1.2k)/10k=-12.02025V befor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 -> SR1 final divider:(90.9k+0R+1.2k)/10k=-11.99675V before IFB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
- R83: value 9.1k 1% -> 0 1%; LCSC C23260 -> C21189; MPN 0603WAF9101T5E -> 0603WAF0000T5E; NOTE Basic negative divider:(82k+9.1k+1.2k)/10k=-12.02025V befor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 -> SR1 final divider:(90.9k+0R+1.2k)/10k=-11.99675V before IFB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
Connections:
- net GND: now also C73.2, C74.2
- net N12: now also C73.1
- net NRAW: now also C74.1
Other:
- note added: "R72=90.9k 0.1%, R83=0R, R73=1.2k 1%, R74=10k 0.1% -> -11.99675V nominal. C62 DNP (pads retained): supported without CFF, noise/PSRR tradeoff; no claimed bench cure. D27/D28 discharge paths are NOT isolation or proof of negative0.3V differential compliance. Headroom/temperature/loop/start-stop/reverse-current qualification remains open. No supply current rating."
- note added: "SR2 PRAW +13.519V / NRAW -14.07752V nominal; independent P5 unchanged. Same exact LDOs and N12 precision divider. No rail-synchronous shutdown. PCB remains old/unsynchronized."
- note added: "U12 ANY-OUT 5,6,9,11 GND; 4,8,10,12 float; SENSE3=P12. Both EP21=GND. C12891 banks IN+/OUT+/IN-/OUT- =4/6/5/4; combined DC+AC bias screening only. C60=1u; C61=100n. EN tied to own raw input, no disconnect or tracking promise."
- note removed: "(R72+R83+R73)/R74 =92.3k/10k -> -12.02025V before IFB; 117.5uA nominal divider current (>5uA required). C61 100n: typical ~120ms start, not rail sequencing. C62 10n improves AC; shutdown FB kick remains a test gate. D27/D28 divert reverse current, do NOT block it. SS34 Vf does NOT prove the negative -0.3V differential limit. 800mA aspiration is load-dependent, not a simultaneous rail guarantee. C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"
- note removed: "Raw +13.537080/-13.928806V remain internal. Final +5V is unchanged and bypasses this sheet. Both exposed pads 21 are GND. Exact requested RGWR parts; NOT a +/-1A supply."
- note removed: "U12 ANY-OUT: 5,6,9,11 to GND; 4,8,10,12 float. SENSE3 -> final output. C60 sees approximately +12V. 4/6/4/3 x22u on IN+/OUT+/IN-/OUT-; typical bias + tolerance/temp/aging screen passes. Require >=10u effective at each IN/OUT; >=20u at positive OUT for accuracy conditions."
