File: modules/usb-power/hardware/06_positive_boost.kicad_sch (KiCad schematic)
At the start: 19 parts, among them U14 TPS55340RTER

Commit message: usb-power: substitute L1 -> TMPC1205HP-220MG-D (C357250), L4/L5 -> SLO1040H6R8MTT (C207852)
- L1: new BigModular:L_TMPC1205HP_220M footprint, land identical to SRP1245A
- L4/L5: new BigModular:L_SLO1040H6R8MTT footprint, engineering-defined land
  (3.5x4.0 pads, 5.0 gap, 12.0 overall) pending vendor drawing
- schematic fields (footprint/MPN/LCSC/manufacturer/note) updated in
  03_bucks, 04_bipolar, 06_positive_boost
- generator part records updated; BOM.csv regenerated (only 3 lines changed)
- ERC 0/0 before and after; netlist connectivity unchanged
- PCB and jlcpcb/assembly untouched (routing task follows)
Parts:
- L5: footprint BigModular:L_KOHER_MDA1040 -> BigModular:L_SLO1040H6R8MTT; LCSC C2847552 -> C207852; MPN MDA1040-6R8M -> SLO1040H6R8MTT; Manufacturer KOHERelec -> Sunltech; NOTE Same exact MDA1040-6R8M as L1/L4; height max4.0mm; manufact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 -> Sunltech SLO1040H6R8MTT; 6.8uH +/-20%; DCR22mohm typ/25mohm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
Changed lines of the file:
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@@
 			)
 		)
-		(property "Footprint" "BigModular:L_KOHER_MDA1040"
+		(property "Footprint" "BigModular:L_SLO1040H6R8MTT"
 			(at 160.02 58.42 0)
 			(hide yes)
@@
 			)
 		)
-		(property "Datasheet" "https://wmsc.lcsc.com/wmsc/upload/file/pdf/v2/lcsc/2401281810_KOHERelec-MDA1040-6R8M_C2847552.pdf"
+		(property "Datasheet" "https://datasheet.lcsc.com/datasheet/pdf/4b813f0bd1895de8fff894fc302289d3.pdf?productCode=C207852"
 			(at 160.02 58.42 0)
 			(hide yes)
@@
 			)
 		)
-		(property "MPN" "MDA1040-6R8M"
+		(property "MPN" "SLO1040H6R8MTT"
 			(at 160.02 58.42 0)
 			(hide yes)
@@
 			)
 		)
-		(property "LCSC" "C2847552"
+		(property "LCSC" "C207852"
 			(at 160.02 58.42 0)
 			(hide yes)
@@
 			)
 		)
-		(property "NOTE" "Same exact MDA1040-6R8M as L1/L4; height max4.0mm; manufacturer Isat table11A/typ12.2A exceeds TPS55340 maximum7.75A fault limit; Irms table6.8A/typ7.8A, DCRmax24.5mohm. Not a guaranteed hot-lot minimum. Saturation/thermal and frontside placement verification pending."
+		(property "NOTE" "Sunltech SLO1040H6R8MTT; 6.8uH +/-20%; DCR22mohm typ/25mohm max. Isat typ10A at approx20% L drop/25C; Idc typ7A at approx40C rise. Height4.0mm max. Land engineering-defined, pending vendor drawing: 2 rectangular pads3.5(X)x4.0(Y)mm, 5.0mm gap, 12.0mm overall. Stock4991 observed2026-10-17, not reserved or guaranteed. No guaranteed hot-lot minimum; PCB fit/stack/saturation/thermal qualification pending."
 			(at 160.02 58.42 0)
 			(hide yes)
@@
 			)
 		)
-		(property "Manufacturer" "KOHERelec"
+		(property "Manufacturer" "Sunltech"
 			(at 160.02 58.42 0)
 			(hide yes)
