File: modules/usb-power/hardware/07_output_rails.kicad_sch (KiCad schematic)
At the start: 6 parts, among them J7 Manual IDC wire landing

Commit message: Fix some PCB to Schematic link issue
Changed lines of the file:
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@@
 	(text "Single red D10: FINAL P5 presence only.\nR32 1k; no blink, MCU or all-rail status claim.\nManual harness from J7; 13..16 NC. Never parallel a PSU."
 		(exclude_from_sim no)
-		(at 231.14 121.92 0)
+		(at 246.888 101.346 0)
 		(effects
 			(font
@@
 	)
 	(junction
+		(at 91.44 111.76)
+		(diameter 0)
+		(color 0 0 0 0)
+	)
+	(junction
+		(at 91.44 109.22)
+		(diameter 0)
+		(color 0 0 0 0)
+	)
+	(junction
 		(at 81.28 116.84)
+		(diameter 0)
+		(color 0 0 0 0)
+	)
+	(junction
+		(at 87.63 109.22)
 		(diameter 0)
 		(color 0 0 0 0)
@@
 	)
 	(junction
-		(at 142.24 109.22)
-		(diameter 0)
-		(color 0 0 0 0)
-	)
-	(junction
-		(at 143.51 109.22)
-		(diameter 0)
-		(color 0 0 0 0)
-	)
-	(junction
 		(at 134.62 238.76)
 		(diameter 0)
@@
 	)
 	(junction
-		(at 83.82 109.22)
+		(at 104.14 111.76)
 		(diameter 0)
 		(color 0 0 0 0)
@@
 	)
 	(junction
-		(at 76.2 119.38)
+		(at 104.14 109.22)
 		(diameter 0)
 		(color 0 0 0 0)
 	)
 	(junction
-		(at 85.09 109.22)
+		(at 86.36 119.38)
 		(diameter 0)
 		(color 0 0 0 0)
 	)
-	(junction
-		(at 81.28 109.22)
-		(diameter 0)
-		(color 0 0 0 0)
-	)
 	(no_connect
 		(at 91.44 121.92)
@@
 	(wire
 		(pts
-			(xy 83.82 109.22) (xy 85.09 109.22)
-		)
-		(stroke
-			(width 0)
-			(type default)
-		)
-	)
-	(wire
-		(pts
-			(xy 86.36 114.3) (xy 91.44 114.3)
-		)
-		(stroke
-			(width 0)
-			(type default)
-		)
-	)
-	(wire
-		(pts
-			(xy 76.2 142.24) (xy 127 142.24)
+			(xy 86.36 129.54) (xy 111.76 129.54)
 		)
 		(stroke
@@
 	(wire
 		(pts
+			(xy 104.14 111.76) (xy 104.14 114.3)
+		)
+		(stroke
+			(width 0)
+			(type default)
+		)
+	)
+	(wire
+		(pts
 			(xy 73.66 209.55) (xy 73.66 238.76)
 		)
@@
 	(wire
 		(pts
-			(xy 127 119.38) (xy 127 142.24)
-		)
-		(stroke
-			(width 0)
-			(type default)
-		)
-	)
-	(wire
-		(pts
-			(xy 81.28 99.06) (xy 81.28 109.22)
-		)
-		(stroke
-			(width 0)
-			(type default)
-		)
-	)
-	(wire
-		(pts
-			(xy 104.14 109.22) (xy 142.24 109.22)
+			(xy 111.76 119.38) (xy 111.76 129.54)
+		)
+		(stroke
+			(width 0)
+			(type default)
+		)
+	)
+	(wire
+		(pts
+			(xy 104.14 109.22) (xy 107.95 109.22)
 		)
 		(stroke
@@
 	(wire
 		(pts
-			(xy 85.09 107.95) (xy 85.09 109.22)
-		)
-		(stroke
-			(width 0)
-			(type default)
-		)
-	)
-	(wire
-		(pts
-			(xy 104.14 111.76) (xy 142.24 111.76)
-		)
-		(stroke
-			(width 0)
-			(type default)
-		)
-	)
-	(wire
-		(pts
 			(xy 73.66 238.76) (xy 134.62 238.76)
 		)
@@
 	(wire
 		(pts
-			(xy 142.24 109.22) (xy 142.24 111.76)
-		)
-		(stroke
-			(width 0)
-			(type default)
-		)
-	)
-	(wire
-		(pts
-			(xy 147.32 99.06) (xy 147.32 109.22)
-		)
-		(stroke
-			(width 0)
-			(type default)
-		)
-	)
-	(wire
-		(pts
-			(xy 83.82 101.6) (xy 83.82 107.95)
+			(xy 87.63 101.6) (xy 87.63 109.22)
 		)
 		(stroke
@@
 	(wire
 		(pts
-			(xy 143.51 109.22) (xy 147.32 109.22)
+			(xy 107.95 101.6) (xy 87.63 101.6)
 		)
 		(stroke
@@
 	(wire
 		(pts
-			(xy 86.36 114.3) (xy 86.36 132.08)
-		)
-		(stroke
-			(width 0)
-			(type default)
-		)
-	)
-	(wire
-		(pts
-			(xy 143.51 107.95) (xy 143.51 109.22)
-		)
-		(stroke
-			(width 0)
-			(type default)
-		)
-	)
-	(wire
-		(pts
-			(xy 104.14 114.3) (xy 137.16 114.3)
-		)
-		(stroke
-			(width 0)
-			(type default)
-		)
-	)
-	(wire
-		(pts
-			(xy 142.24 107.95) (xy 143.51 107.95)
-		)
-		(stroke
-			(width 0)
-			(type default)
-		)
-	)
-	(wire
-		(pts
-			(xy 83.82 101.6) (xy 142.24 101.6)
-		)
-		(stroke
-			(width 0)
-			(type default)
-		)
-	)
-	(wire
-		(pts
-			(xy 142.24 101.6) (xy 142.24 107.95)
+			(xy 91.44 109.22) (xy 91.44 111.76)
 		)
 		(stroke
@@
 	(wire
 		(pts
-			(xy 85.09 109.22) (xy 91.44 109.22)
-		)
-		(stroke
-			(width 0)
-			(type default)
-		)
-	)
-	(wire
-		(pts
 			(xy 78.74 106.68) (xy 91.44 106.68)
 		)
@@
 	(wire
 		(pts
-			(xy 132.08 116.84) (xy 132.08 137.16)
+			(xy 114.3 116.84) (xy 114.3 133.35)
 		)
 		(stroke
@@
 	(wire
 		(pts
-			(xy 83.82 109.22) (xy 83.82 111.76)
-		)
-		(stroke
-			(width 0)
-			(type default)
-		)
-	)
-	(wire
-		(pts
-			(xy 137.16 114.3) (xy 137.16 132.08)
-		)
-		(stroke
-			(width 0)
-			(type default)
-		)
-	)
-	(wire
-		(pts
 			(xy 104.14 106.68) (xy 152.4 106.68)
 		)
@@
 	(wire
 		(pts
-			(xy 104.14 116.84) (xy 132.08 116.84)
-		)
-		(stroke
-			(width 0)
-			(type default)
-		)
-	)
-	(wire
-		(pts
-			(xy 142.24 109.22) (xy 143.51 109.22)
-		)
-		(stroke
-			(width 0)
-			(type default)
-		)
-	)
-	(wire
-		(pts
-			(xy 81.28 109.22) (xy 83.82 109.22)
+			(xy 104.14 116.84) (xy 114.3 116.84)
+		)
+		(stroke
+			(width 0)
+			(type default)
+		)
+	)
+	(wire
+		(pts
+			(xy 104.14 109.22) (xy 104.14 111.76)
+		)
+		(stroke
+			(width 0)
+			(type default)
+		)
+	)
+	(wire
+		(pts
+			(xy 87.63 109.22) (xy 91.44 109.22)
+		)
+		(stroke
+			(width 0)
+			(type default)
+		)
+	)
+	(wire
+		(pts
+			(xy 107.95 109.22) (xy 107.95 101.6)
 		)
 		(stroke
@@
 	(wire
 		(pts
-			(xy 81.28 137.16) (xy 132.08 137.16)
+			(xy 81.28 133.35) (xy 114.3 133.35)
 		)
 		(stroke
@@
 	(wire
 		(pts
-			(xy 40.64 119.38) (xy 76.2 119.38)
-		)
-		(stroke
-			(width 0)
-			(type default)
-		)
-	)
-	(wire
-		(pts
-			(xy 81.28 99.06) (xy 147.32 99.06)
-		)
-		(stroke
-			(width 0)
-			(type default)
-		)
-	)
-	(wire
-		(pts
-			(xy 83.82 107.95) (xy 85.09 107.95)
-		)
-		(stroke
-			(width 0)
-			(type default)
-		)
-	)
-	(wire
-		(pts
-			(xy 86.36 132.08) (xy 137.16 132.08)
+			(xy 40.64 119.38) (xy 91.44 119.38)
 		)
 		(stroke
@@
 	(wire
 		(pts
-			(xy 81.28 116.84) (xy 81.28 137.16)
+			(xy 81.28 116.84) (xy 81.28 133.35)
 		)
 		(stroke
@@
 	(wire
 		(pts
-			(xy 104.14 119.38) (xy 127 119.38)
-		)
-		(stroke
-			(width 0)
-			(type default)
-		)
-	)
-	(wire
-		(pts
-			(xy 83.82 111.76) (xy 91.44 111.76)
-		)
-		(stroke
-			(width 0)
-			(type default)
-		)
-	)
-	(wire
-		(pts
-			(xy 76.2 119.38) (xy 91.44 119.38)
+			(xy 104.14 119.38) (xy 111.76 119.38)
 		)
 		(stroke
@@
 	(wire
 		(pts
-			(xy 25.4 109.22) (xy 81.28 109.22)
+			(xy 55.88 109.22) (xy 87.63 109.22)
 		)
 		(stroke
@@
 	(wire
 		(pts
-			(xy 76.2 119.38) (xy 76.2 142.24)
+			(xy 86.36 119.38) (xy 86.36 129.54)
+		)
+		(stroke
+			(width 0)
+			(type default)
+		)
+	)
+	(wire
+		(pts
+			(xy 91.44 111.76) (xy 91.44 114.3)
 		)
 		(stroke
@@
 	(label "LED_P_A"
 		(at 289.56 88.9 0)
-		(effects
-			(font
-				(size 0.95 0.95)
-			)
-			(justify left bottom)
-		)
-	)
-	(label "GND"
-		(at 111.76 132.08 0)
 		(effects
 			(font
@@
 	(hierarchical_label "GND"
 		(shape passive)
-		(at 25.4 109.22 180)
+		(at 55.88 109.22 180)
 		(effects
 			(font
@@
 		)
 		(property "Value" "Manual IDC wire landing"
-			(at 96.52 103.22 0)
-			(show_name no)
-			(do_not_autoplace no)
+			(at 97.282 92.964 0)
+			(show_name no)
+			(do_not_autoplace no)

Commit message: Add more space for usb-power IDC socket and -12V now stays on the bottom.
Parts:
- J7: value Manual IDC wire landing -> IDC 2x8 box header; footprint BigModular:WireLanding_2x08_P2.54mm -> BigModular:IDC-Header_2x08_P2.54mm_Vertical; NOTE ON-CARRIER numbered solder lands, not an extra purchasable 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 -> Hand-soldered 2x8 shrouded IDC box header (Eurorack 16-pin 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
Changed lines of the file:
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@@
 			)
 		)
-		(property "Value" "Manual IDC wire landing"
+		(property "Value" "IDC 2x8 box header"
 			(at 97.282 92.964 0)
 			(show_name no)
@@
 			)
 		)
-		(property "Footprint" "BigModular:WireLanding_2x08_P2.54mm"
+		(property "Footprint" "BigModular:IDC-Header_2x08_P2.54mm_Vertical"
 			(at 96.52 114.3 0)
 			(hide yes)
@@
 			)
 		)
-		(property "NOTE" "ON-CARRIER numbered solder lands, not an extra purchasable box header. Physical output cable boundary; single output, never another active source."
+		(property "NOTE" "Hand-soldered 2x8 shrouded IDC box header (Eurorack 16-pin power cable). Pin 1/2 = -12 V toward module bottom. Single output, never another active source."
 			(at 96.52 114.3 0)
 			(hide yes)
