File: modules/usb-power/hardware/usb-power.kicad_pcb (KiCad board)
At the start: 4 copper layers, 100.5 x 30 mm, 120 parts, among them J1 TYPE-C-31-M-12, J7 Manual IDC wire landing, SW1 TL3340AF160QG, U1 CH224A, U12 TPS7A4700RGWR, U13 TPS7A3301RGWR, U14 TPS55340RTER, U2 TPS26600PWPR, U3 TPS54302DDCR, U5 TPS54302DDCR

Commit message: Add testing pad in the bottom of the PCB.
Routing:
- net /GND: track 191.5 -> 193.4 mm
- net /USB PD input/USB_VBUS: track 20.6 -> 22.2 mm
- net /VPROT: track 239.5 -> 241.1 mm
- net /Direct 9V negative IBB/NRAW: track 220.2 -> 221.8 mm
- net /VIN9: track 52.0 -> 53.6 mm
- net /Direct 9V positive boost/PRAW: track 112.3 -> 113.9 mm
Other:
- board text added: "GND"
- board text added: "N12"
- board text added: "NC"
- board text added: "P12"
- board text added: "P5"
- board text added: "TP GND"
- board text added: "TP NRAW"
- board text added: "TP PRAW"
- board text added: "TP VBUS"
- board text added: "TP VIN9"
- board text added: "TP VPROT"

Commit message: Add some final optimizations before FAB.
Parts:
- moved C88 0.80 mm to (127.0, 83.7)
- moved C61 0.50 mm to (64.0, 82.6)
- moved C36 0.40 mm to (108.4, 92.6)
- moved C7 0.40 mm to (129.0, 99.3), turned to -90 degrees
- moved R6 0.25 mm to (76.8, 87.1)
Routing:
- net /GND: track 193.4 -> 197.6 mm
- net /Direct 9V negative IBB/NRAW: track 221.8 -> 225.5 mm
- net /P5: track 68.7 -> 70.9 mm
- net /Autonomous hardware window and retry/OV_SET: track 7.67 -> 9.13 mm
- net /Independent +5V buck/FIVE_SW: track 9.92 -> 11.3 mm
- net /N12: track 80.1 -> 81.4 mm
- net /Autonomous hardware window and retry/EF_MODE: track 11.8 -> 12.9 mm
- net /VIN9: track 53.6 -> 52.9 mm, vias 10 -> 9
- net /VPROT: track 241.1 -> 240.5 mm, vias 31 -> 29

Commit message: Add more space for usb-power IDC socket and -12V now stays on the bottom.
Parts:
- removed the ? at (79.2, 77.3)
- removed the ? at (106.2, 77.3)
- J7: value Manual IDC wire landing -> IDC 2x8 box header; footprint BigModular:WireLanding_2x08_P2.54mm -> BigModular:IDC-Header_2x08_P2.54mm_Vertical
- moved J7 18.4 mm to (101.5, 72.6), turned to -90 degrees
Routing:
- net /N12: track 81.4 -> 103.6 mm
- net /GND: track 197.6 -> 216.0 mm, vias 113 -> 116
- net /P5: track 70.9 -> 79.5 mm
- net /P12: track 58.0 -> 61.5 mm
Other:
- board size 100.5 x 30 mm -> 100.5 x 35 mm
