File: modules/midi/hardware/midi.kicad_sch (KiCad schematic)
At the start: 47 parts, among them J1 PJ366ST, J10 Eurorack_2x5, J11 UPDI, J2 PJ301M-12, J3 PJ301M-12, J4 PJ301M-12, J5 PJ301M-12, J6 PJ301M-12, J7 PJ301M-12, J8 PJ301M-12, J9 PJ301M-12, U1 ATtiny1616-MNR, U3 HT7550-1

Commit message: midi: move regulator group beside power header, add U3 heat-sink copper (R2)
- Relocate U3/R20/C4/C5/D10 to the open area right of J10, outside the
  16-pin IDC overhang; J11/R11 to the strip left of J10.
- Split GND pours on both layers around VIN_LDO heat-sink copper for U3
  (~285 mm2 total, 9 heat vias); heat stays at the bottom edge.
- Re-route power chain, UPDI and +5V trunk; GND returns on B.Cu.
- Re-export JLCPCB carrier (BOM identical, 6 placements moved, +4 via holes),
  refresh DRC/ERC records and 3D fit renders.
- Update research.md, mechanics.md, Code.md, README, AGENTS and jlcpcb/README.

Checks: ERC 0, DRC 0, unconnected 0, schematic parity 0, manifest equal.
Parts:
- C1: LCSC (none) -> C14663; MPN (none) -> CC0603KRX7R9BB104; Manufacturer (none) -> YAGEO; Voltage 16V -> 50V
- C3, C4: LCSC (none) -> C15850; MPN (none) -> CL21A106KAYNNNE; Manufacturer (none) -> Samsung; Voltage 16V -> 25V
- C5: LCSC (none) -> C28323; MPN (none) -> CL21B105KBFNNNE; Manufacturer (none) -> Samsung; Voltage 25V -> 50V
- D10: MPN (none) -> B5819W SL; Manufacturer (none) -> CJ (Jiangsu Changjing)
- R10, R12, R13, R14, R15, R16, R17, R18, R19, R3, R4, R5, R6, R7, R8, R9: LCSC (none) -> C21190; MPN (none) -> 0603WAF1001T5E; Manufacturer (none) -> UNI-ROYAL
- R11, R21: LCSC (none) -> C23162; MPN (none) -> 0603WAF4701T5E; Manufacturer (none) -> UNI-ROYAL
- R2: LCSC (none) -> C31850; MPN (none) -> 0603WAF2202T5E; Manufacturer (none) -> UNI-ROYAL
- R20: LCSC (none) -> C414944; MPN (none) -> HP06W2F390JT5E; Manufacturer (none) -> UNI-ROYAL; Note Dropper: shares LDO heat in the ~77 mA worst case (research 3.1) -> Dropper: shares LDO heat in the ~77 mA worst case (research 3.1); anti-surge 0.5 W part, sits on the VIN_LDO heat-sink copper; Power 0.25W -> 0.5W
- U1: MPN (none) -> ATTINY1616-MNR; Manufacturer (none) -> Microchip
- U3: MPN (none) -> HT7550-1; Manufacturer (none) -> Holtek; Note 30 V max input, 150 mA -> 30 V max input, 150 mA. Tab = pin 2 (VIN): heat-sink copper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

Commit message: Remove R21 divider and keep everything same as Bread Modular's version.
Parts:
- removed R2: 22k, MIDI:R_0603_1608Metric, symbol MIDI:R
- removed R21: 4.7k, MIDI:R_0603_1608Metric, symbol MIDI:R
- JP1: Note 1x3 2.54 mm header + shunt. 1-2 = Type A (Tip = data), 2-3 = Type B (Ring = data). No shunt = no input -> 1x3 2.54 mm header + shunt. 1-2 = Type A (Tip = data), 2-3 = Type B (Ring = data). No shunt = no input. Common drives PB3 directly, as Bread Modular V1 (no series R, no pull-up)
Connections:
- net DATA is gone; now on net RX: JP1.2 (C)
Other:
- note added: "BIG MODULAR MIDI - S4 schematic (5 V logic, BM V1 direct input). Circuit intent: docs/research.md"
- note removed: "BIG MODULAR MIDI - S3 schematic (5 V logic). Circuit intent: docs/research.md"
