File: modules/audio-out/hardware/audio-out.kicad_pcb (KiCad board)
At the start: 2 copper layers, 19 x 110 mm, 33 parts, among them J1 PJ301M-12, J2 PJ301M-12, J3 PJ366ST, J4 PJ366ST, J5 Eurorack_2x5, U1 OPA1678IDR, U2 MC33178DR2G

Commit message: Update the audio out module.
Parts:
- moved R9 0.67 mm to (109.8, 122.0)
- moved C9 0.50 mm to (104.1, 119.4)
Routing:
- net /+12V: track 107.5 -> 107.0 mm
