File: modules/midi/hardware/v1/midi.kicad_pcb (KiCad board)
At the start: 2 copper layers, 19 x 110 mm, 45 parts, among them J1 PJ366ST, J10 Eurorack_2x5, J11 UPDI, J2 PJ301M-12, J3 PJ301M-12, J4 PJ301M-12, J5 PJ301M-12, J6 PJ301M-12, J7 PJ301M-12, J8 PJ301M-12, J9 PJ301M-12, U1 ATtiny1616-MNR, U3 HT7550-1

Commit message: Add LED drivers for MIDI module.
Parts:
- added Q11: MMBT3904, MIDI:SOT-23, B.Cu at (117.3, 71.0)
- added Q12: MMBT3904, MIDI:SOT-23, B.Cu at (117.3, 81.0)
- added Q13: MMBT3904, MIDI:SOT-23, B.Cu at (117.3, 91.5)
- added Q14: MMBT3904, MIDI:SOT-23, B.Cu at (117.3, 102.0)
- added Q15: MMBT3904, MIDI:SOT-23, B.Cu at (117.3, 112.5)
- added Q16: MMBT3904, MIDI:SOT-23, B.Cu at (117.3, 123.0)
- added Q17: MMBT3904, MIDI:SOT-23, B.Cu at (117.3, 133.4)
- added Q18: MMBT3904, MIDI:SOT-23, B.Cu at (117.3, 143.9)
- added R31: 10k, MIDI:R_0603_1608Metric, B.Cu at (113.5, 72.0)
- added R32: 10k, MIDI:R_0603_1608Metric, B.Cu at (113.5, 82.5)
- added R33: 10k, MIDI:R_0603_1608Metric, B.Cu at (113.5, 93.0)
- added R34: 10k, MIDI:R_0603_1608Metric, B.Cu at (115.6, 108.0)
- added R35: 10k, MIDI:R_0603_1608Metric, B.Cu at (113.5, 116.0)
- added R36: 10k, MIDI:R_0603_1608Metric, B.Cu at (113.5, 124.5)
- added R37: 10k, MIDI:R_0603_1608Metric, B.Cu at (113.5, 135.0)
- added R38: 10k, MIDI:R_0603_1608Metric, B.Cu at (113.5, 145.5)
- moved D7 2.54 mm to (117.2, 138.2), turned to -90 degrees
- moved D8 2.54 mm to (117.2, 148.7), turned to -90 degrees
- moved D6 2.54 mm to (117.2, 127.7), turned to -90 degrees
- moved D1 2.54 mm to (117.2, 75.2), turned to -90 degrees
- moved D2 2.54 mm to (117.2, 85.7), turned to -90 degrees
- moved D3 2.54 mm to (117.2, 96.2), turned to -90 degrees
- moved D4 2.54 mm to (117.2, 106.7), turned to -90 degrees
- moved D5 2.54 mm to (117.2, 117.2), turned to -90 degrees
- moved R4 1.00 mm to (117.3, 73.6), turned to 0 degrees
- moved R10 0.51 mm to (117.3, 104.6), turned to 0 degrees
- moved R13 0.51 mm to (117.3, 115.1), turned to 0 degrees
- moved R15 0.51 mm to (117.3, 125.6), turned to 0 degrees
- moved R17 0.51 mm to (117.3, 136.1), turned to 0 degrees
- moved R19 0.51 mm to (117.3, 146.6), turned to 0 degrees
- moved R6 0.51 mm to (117.3, 83.6), turned to 0 degrees
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Connections:
- net /OUT1 renamed /CH1/OUT
- net /OUT2 renamed /CH2/OUT
- net /OUT3 renamed /CH3/OUT
- net /OUT4 renamed /CH4/OUT
- net /OUT5 renamed /CH5/OUT
- net /OUT6 renamed /CH6/OUT
- net /OUT7 renamed /CH7/OUT
- net /OUT8 renamed /CH8/OUT
- D1 pad 1: /GND -> /CH1/LED_K
- D1 pad 2: /LED1_A -> /+5V
- D2 pad 1: /GND -> /CH2/LED_K
- D2 pad 2: /LED2_A -> /+5V
- D3 pad 1: /GND -> /CH3/LED_K
- D3 pad 2: /LED3_A -> /+5V
- D4 pad 1: /GND -> /CH4/LED_K
- D4 pad 2: /LED4_A -> /+5V
- D5 pad 1: /GND -> /CH5/LED_K
- D5 pad 2: /LED5_A -> /+5V
- D6 pad 1: /GND -> /CH6/LED_K
- D6 pad 2: /LED6_A -> /+5V
- D7 pad 1: /GND -> /CH7/LED_K
- D7 pad 2: /LED7_A -> /+5V
- D8 pad 1: /GND -> /CH8/LED_K
- D8 pad 2: /LED8_A -> /+5V
- R10 pad 1: /CH4_LED -> /CH4/LED_K
- R10 pad 2: /LED4_A -> /CH4/Q_C
- R13 pad 1: /CH5_LED -> /CH5/LED_K
- R13 pad 2: /LED5_A -> /CH5/Q_C
- R15 pad 1: /CH6_LED -> /CH6/LED_K
- R15 pad 2: /LED6_A -> /CH6/Q_C
- R17 pad 1: /CH7_LED -> /CH7/LED_K
- R17 pad 2: /LED7_A -> /CH7/Q_C
- R19 pad 1: /CH8_LED -> /CH8/LED_K
- R19 pad 2: /LED8_A -> /CH8/Q_C
- R4 pad 1: /CH1_LED -> /CH1/LED_K
- R4 pad 2: /LED1_A -> /CH1/Q_C
- R6 pad 1: /CH2_LED -> /CH2/LED_K
- R6 pad 2: /LED2_A -> /CH2/Q_C
- R8 pad 1: /CH3_LED -> /CH3/LED_K
- R8 pad 2: /LED3_A -> /CH3/Q_C
Routing:
- net /+5V: track 64.2 -> 221.7 mm
- net /GND: track 18.8 -> 35.1 mm, vias 17 -> 18
- net /CH5_LED: track 10.7 -> 3.34 mm
- net /CH4_LED: track 18.1 -> 11.0 mm
- net /CH4/Q_B: track 0.00 -> 5.04 mm
- net /CH3_LED: track 28.2 -> 23.5 mm
- net /CH2_LED: track 38.3 -> 33.6 mm
- net /CH1_LED: track 48.4 -> 43.7 mm
- net /CH5/Q_B: track 0.00 -> 4.64 mm
- net /CH8_LED: track 39.7 -> 35.1 mm
- net /CH7_LED: track 27.3 -> 23.0 mm
- net /CH6_LED: track 16.1 -> 11.8 mm
- net /CH7/Q_C: track 0.00 -> 2.65 mm
- net /CH8/Q_C: track 0.00 -> 2.65 mm
- net /CH6/Q_C: track 0.00 -> 2.65 mm
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