File: modules/imix/hardware/imix.kicad_pcb (KiCad board)
At the start: 2 copper layers, 29 x 110 mm, 46 parts, among them J1 PJ301M-12, J10 Eurorack_2x5, J2 PJ301M-12, J3 PJ301M-12, J4 PJ301M-12, J5 PJ301M-12, U1 TL072CDT, U2 TL072CDT, U3 TL072CDT

Commit message: Set proper output resistors to match with the voltage.
Parts:
- R18: footprint IMIX:R_1206_3216Metric -> IMIX:R_2512_6332Metric
- moved R18 3.20 mm to (108.9, 144.0)
Routing:
- net /MIX: track 8.32 -> 7.47 mm
