File: modules/imix/hardware/imix.kicad_sch (KiCad schematic)
At the start: 46 parts, among them J1 PJ301M-12, J10 Eurorack_2x5, J2 PJ301M-12, J3 PJ301M-12, J4 PJ301M-12, J5 PJ301M-12, U1 TL072CDT, U2 TL072CDT, U3 TL072CDT

Commit message: Set proper output resistors to match with the voltage.
Parts:
- R18: footprint IMIX:R_1206_3216Metric -> IMIX:R_2512_6332Metric; LCSC C4410 -> C54315; MPN 1206W4F1001T5E -> 25121WF1001T4E; Note Output series / short-circuit protection; 1206 (250 mW): ~1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 -> Output series / short-circuit and mis-patch protection; 251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
Changed lines of the file:
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@@
 			)
 		)
-		(property "Footprint" "IMIX:R_1206_3216Metric"
+		(property "Footprint" "IMIX:R_2512_6332Metric"
 			(at 193.04 193.04 90)
 			(hide yes)
@@
 			)
 		)
-		(property "Note" "Output series / short-circuit protection; 1206 (250 mW): ~110 mW with a +/-10.5 V output shorted"
+		(property "Note" "Output series / short-circuit and mis-patch protection; 2512 (1 W): ~0.51 W with a -12 V source on MIX against +10.5 V"
 			(at 193.04 193.04 90)
 			(hide yes)
@@
 			)
 		)
-		(property "LCSC" "C4410"
+		(property "LCSC" "C54315"
 			(at 193.04 193.04 90)
 			(hide yes)
@@
 			)
 		)
-		(property "MPN" "1206W4F1001T5E"
+		(property "MPN" "25121WF1001T4E"
 			(at 193.04 193.04 90)
 			(hide yes)
