File: modules/8bit/hardware/8bit.kicad_pcb (KiCad board)
At the start: 2 copper layers, 19 x 110 mm, 48 parts, among them J1 PJ301M-12, J2 PJ301M-12, J3 PJ301M-12, J4 Eurorack_2x5, J5 UPDI, Q1 MMBT3904, SW1 MODE, U1 ATtiny1616-MNR, U2 HT7550-1, U3 TL072, U4 MCP6001

Commit message: Update the 8bit switch to a DIP version.
Parts:
- SW1: footprint 8BIT:K2-1808SN-A4SW-01 -> 8BIT:SW_PUSH_6mm_H7.3mm
- moved C14 8.10 mm to (105.1, 128.6)
- moved R10 7.40 mm to (102.6, 127.6)
- moved R11 7.40 mm to (102.6, 131.0)
- moved SW1 3.91 mm to (110.2, 139.2)
Routing:
- net /VREF_DIV: track 19.8 -> 28.2 mm
- net /BUTTON: track 74.1 -> 73.3 mm
- net GND: vias 15 -> 16
Other:
- board text added: "8BIT S5"
- board text removed: "8BIT S4"
