File: modules/mcc/hardware/mcc.kicad_pcb (KiCad board)
At the start: 2 copper layers, 29 x 110 mm, 68 parts, among them J1 PJ301M-12, J11 PJ301M-12, J12 PJ301M-12, J13 PJ301M-12, J14 PJ301M-12, J2 PJ301M-12, J3 Eurorack_2x5, J4 UPDI, Q1 MMBT3904, SW1 BANK, U1 ATtiny1616-MNR, U2 HT7550-1, U3 CJ431, U4 MCP6002, U5 MCP6002

Commit message: Improve MCC.
Parts:
- R4: footprint MCC:R_0805_2012Metric -> MCC:R_1206_3216Metric
- moved R4 0.50 mm to (118.8, 62.1)
Other:
- board text added: "MCC V1"
- board text removed: "MCC S2"
