File: modules/16bit/panels/front-pcb/16bit-panel.kicad_pcb (KiCad board)
At the start: 2 copper layers, 30 x 128.5 mm, 13 parts

Commit message: 16bit: start manual re-route; place and route bottom power/output stage
- Strip R1 router copper; move SMD parts off-board for hand placement
- 4-layer stackup (F sig / In1 GND / In2 +3V3 / B sig), Power net class
- Move CV jacks/pots up and to the edge, bottom pots RV3/RV4 to Y128
  (board, panel, geometry.json) to free the middle for the RP2350
- Place and route J6 entry, D2/D3, U8/U9 regulators, U5 output amps,
  VREF divider and outputs to J4/J5 (B.Cu + F.Cu only, no vias in pads)
- Document the no-vias-in-SMD-pads rule for the manual route

Native DRC + schematic parity: 0 violations, 0 parity issues.

Co-Authored-By: Claude Opus 5.5 <noreply@anthropic.com>
Parts:
- moved H4 5.39 mm to (105.5, 82.0)
- moved H5 5.39 mm to (124.5, 82.0)
- moved H8 5.00 mm to (107.5, 98.5)
- moved H9 5.00 mm to (122.5, 98.5)
- moved H10 2.00 mm to (107.5, 127.5)
- moved H11 2.00 mm to (122.5, 127.5)
