File: modules/32bit/hardware/32bit.kicad_pcb (KiCad board)
At the start: 4 copper layers, 29 x 110 mm, 103 parts, among them J1 PJ301M-12, J2 PJ301M-12, J3 PJ301M-12, J4 PJ301M-12, J5 PJ301M-12, J6 Eurorack_2x5, J7 USB-C, J8 PJ301M-12, J9 PJ301M-12, Q1 MMBT3904, SW1 MODE, SW2 BOOT, SW3 RESET, U1 ESP32-S3-WROOM-1U-N16R8, U4 ES8388, U5 TL072, U6 MCP6002, U7 TL074, U8 AMS1117-5.0, U9 AMS1117-3.3

Commit message: 32bit: R1 manual routing complete
ESP32 moved left with U6 and the ES8388 codec beside it; CV ADC on IO1/IO2,
I2C on IO38/IO39, codec inputs LIN2/RIN2 (logged in docs/firmware-pins.md).
All nets routed by hand: DRC 0 / unconnected 0 / parity 0, no vias in SMD
pads, In1/In2 planes one piece. Right-edge parts nudged toward 1 mm edge
clearance where possible; board rule stays 0.5 mm.

Co-Authored-By: Claude Opus 5.5 <noreply@anthropic.com>
Parts:
- R43, R47: footprint 32BIT:R_0603_1608Metric -> 32BIT:R_0402_1005Metric
- moved D4 98.9 mm to (107.5, 72.6)
- moved FB1 91.7 mm to (102.4, 149.4), turned to 90 degrees
- moved R55 83.3 mm to (127.8, 150.3), turned to 90 degrees
- moved C7 82.0 mm to (102.6, 153.6)
- moved C8 80.8 mm to (102.6, 154.6)
- moved C5 78.0 mm to (102.3, 143.4)
- moved C6 77.6 mm to (102.4, 145.4), turned to -90 degrees
- moved R4 75.6 mm to (102.6, 152.5), turned to 0 degrees
- moved R20 52.0 mm to (125.0, 166.6), turned to 0 degrees
- moved R47 51.5 mm to (122.8, 133.9), turned to -90 degrees
- moved C40 49.3 mm to (121.9, 135.6), turned to 0 degrees
- moved R43 49.0 mm to (121.8, 133.9), turned to -90 degrees
- moved C41 47.2 mm to (124.1, 134.0), turned to -90 degrees
- moved C38 47.0 mm to (126.2, 134.0), turned to -90 degrees
- moved C39 46.2 mm to (125.1, 134.0), turned to -90 degrees
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Connections:
- R21 pad 1: +3V3_8388 -> +3V3
- R22 pad 1: +3V3_8388 -> +3V3
- U1 pad 17: /CV1_ADC -> unconnected-(U1-IO9-Pad17)
- U1 pad 18: /CV2_ADC -> unconnected-(U1-IO10-Pad18)
- U1 pad 24: /CCLK -> unconnected-(U1-IO47-Pad24)
- U1 pad 25: /CDATA -> unconnected-(U1-IO48-Pad25)
- U1 pad 31: unconnected-(U1-IO38-Pad31) -> /CCLK
- U1 pad 32: unconnected-(U1-IO39-Pad32) -> /CDATA
- U1 pad 38: unconnected-(U1-IO2-Pad38) -> /CV2_ADC
- U1 pad 39: unconnected-(U1-IO1-Pad39) -> /CV1_ADC
- U4 pad 21: unconnected-(U4-RIN2-Pad21) -> /CODEC_RIN
- U4 pad 22: unconnected-(U4-LIN2-Pad22) -> /CODEC_LIN
- U4 pad 23: /CODEC_RIN -> unconnected-(U4-RIN1-Pad23)
- U4 pad 24: /CODEC_LIN -> unconnected-(U4-LIN1-Pad24)
Routing:
- net /EN: track 0.00 -> 127.5 mm, vias 0 -> 3
- net /MIDI_RX: track 0.00 -> 101.3 mm, vias 0 -> 2
- net /BOOT: track 0.00 -> 96.9 mm, vias 0 -> 2
- net /USB_DP: track 0.00 -> 88.3 mm, vias 0 -> 2
- net /USB_DM: track 0.00 -> 87.9 mm, vias 0 -> 2
- net +12V_F: track 15.1 -> 98.7 mm, vias 1 -> 3
- net /LED: track 0.00 -> 65.2 mm, vias 0 -> 2
- net /CODEC_LIN: track 10.6 -> 68.8 mm, vias 0 -> 2
- net -12V_F: track 44.1 -> 95.8 mm
- net /CV1_BUF: track 14.8 -> 63.7 mm, vias 0 -> 2
- net /BUTTON: track 0.00 -> 43.1 mm, vias 0 -> 1
- net /CODEC_RIN: track 13.2 -> 55.9 mm
- net /CODEC_LOUT: track 2.70 -> 35.2 mm, vias 1 -> 2
- net +5V: track 0.00 -> 31.2 mm, vias 0 -> 4
- net /CV1_IN: track 61.2 -> 30.6 mm
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- added copper zone on B.Cu, net +5V
- added copper zone on F.Cu, net +5V
