File: modules/32bit/hardware/32bit.kicad_pcb (KiCad board)
At the start: 4 copper layers, 29 x 110 mm, 103 parts, among them J1 PJ301M-12, J2 PJ301M-12, J3 PJ301M-12, J4 PJ301M-12, J5 PJ301M-12, J6 Eurorack_2x5, J7 USB-C, J8 PJ301M-12, J9 PJ301M-12, Q1 MMBT3904, SW1 MODE, SW2 BOOT, SW3 RESET, U1 ESP32-S3-WROOM-1U-N16R8, U4 ES8388, U5 TL072, U6 MCP6002, U7 TL074, U8 AMS1117-5.0, U9 AMS1117-3.3

Commit message: Make sure 32bit Fab Ready
Parts:
- moved C29 10.7 mm to (113.0, 86.6)
- moved C3 9.87 mm to (110.5, 97.6), turned to 180 degrees
- moved R3 6.71 mm to (119.0, 71.0), turned to -90 degrees
- moved C4 5.56 mm to (124.6, 106.8), turned to 180 degrees
- moved D6 5.16 mm to (122.5, 115.5), turned to 180 degrees
- moved R18 4.60 mm to (119.4, 116.1), turned to 180 degrees
- moved R15 4.55 mm to (104.4, 116.1), turned to 180 degrees
- moved C7 4.49 mm to (101.5, 149.2), turned to -90 degrees
- moved R55 4.40 mm to (127.9, 145.9), turned to -90 degrees
- moved R41 3.73 mm to (109.5, 78.9), turned to -90 degrees
- moved R45 3.70 mm to (120.4, 78.9), turned to -90 degrees
- moved C8 3.57 mm to (101.5, 151.2), turned to 90 degrees
- moved R14 3.15 mm to (107.5, 112.8)
- moved R17 3.15 mm to (122.5, 112.8)
- moved C1 3.05 mm to (105.4, 106.8), turned to 180 degrees
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Routing:
- net /MIDI_IN: track 9.44 -> 17.3 mm
- net +5V: track 31.2 -> 38.5 mm
- net /CODEC_ROUT: track 24.7 -> 17.9 mm
- net GND: track 71.9 -> 68.3 mm, vias 29 -> 38
- net Net-(U7D--): track 3.26 -> 6.12 mm
- net /IN_R: track 2.65 -> 5.16 mm
- net +3V3: track 23.6 -> 21.1 mm, vias 15 -> 18
- net /IN_L: track 2.65 -> 5.11 mm
- net /EN: track 127.5 -> 129.9 mm
- net /MIDI_RX: track 101.3 -> 99.5 mm, vias 2 -> 4
- net +12V: track 5.95 -> 7.72 mm
- net Net-(U5B-+): track 10.6 -> 8.90 mm
- net Net-(U7C--): track 3.26 -> 4.87 mm
- net /CODEC_LIN: track 68.8 -> 67.3 mm
- net /CODEC_RIN: track 55.9 -> 54.4 mm
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
Commit message: Add standard UPDI labels for 32bit to hats.
Other:
- board text added: "D"
- board text added: "P"
Changed lines of the file:
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@@
 	)
 	(embedded_fonts no)
+	(gr_text "P"
+		(at 106.85 66.75 0)
+		(layer "B.SilkS")
+		(effects
+			(font
+				(size 1 1)
+				(thickness 0.15)
+			)
+			(justify mirror)
+		)
+	)
+	(gr_text "D"
+		(at 113.15 66.75 0)
+		(layer "B.SilkS")
+		(effects
+			(font
+				(size 1 1)
+				(thickness 0.15)
+			)
+			(justify mirror)
+		)
+	)
 )
