File: modules/32bit/hardware/32bit.kicad_sch (KiCad schematic)
At the start: 103 parts, among them J1 PJ301M-12, J2 PJ301M-12, J3 PJ301M-12, J4 PJ301M-12, J5 PJ301M-12, J6 Eurorack_2x5, J7 USB-C, J8 PJ301M-12, J9 PJ301M-12, Q1 MMBT3904, SW1 MODE, SW2 BOOT, SW3 RESET, U1 ESP32-S3-WROOM-1U-N16R8, U4 ES8388, U5 TL072, U6 MCP6002, U7 TL074, U8 AMS1117-5.0, U9 AMS1117-3.3

Commit message: 32bit: R1 manual routing complete
ESP32 moved left with U6 and the ES8388 codec beside it; CV ADC on IO1/IO2,
I2C on IO38/IO39, codec inputs LIN2/RIN2 (logged in docs/firmware-pins.md).
All nets routed by hand: DRC 0 / unconnected 0 / parity 0, no vias in SMD
pads, In1/In2 planes one piece. Right-edge parts nudged toward 1 mm edge
clearance where possible; board rule stays 0.5 mm.

Co-Authored-By: Claude Opus 5.5 <noreply@anthropic.com>
Parts:
- R21: Note I2C CDATA pull-up (Bread Modular R24) -> I2C CDATA pull-up to +3V3 (Bread Modular R24: +3V3_8388; R1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
- R22: Note I2C CCLK pull-up (Bread Modular R25) -> I2C CCLK pull-up to +3V3 (Bread Modular R25: +3V3_8388; R1 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
- R43, R47: footprint 32BIT:R_0603_1608Metric -> 32BIT:R_0402_1005Metric; LCSC C25803 -> C25741; MPN 0603WAF1003T5E -> 0402WGF1003TCE; Note Input bias to VMID (Bread Modular R19/R16) -> Input bias to VMID (Bread Modular R19/R16); 0402 to fit bes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
Connections:
- net +3V3: now also R21.1, R22.1
- net +3V3_8388: no longer R21.1, R22.1
- net CCLK: now also U1.31 (IO38); no longer U1.24 (IO47)
- net CDATA: now also U1.32 (IO39); no longer U1.25 (IO48)
- net CODEC_LIN: now also U4.22 (LIN2); no longer U4.24 (LIN1)
- net CODEC_RIN: now also U4.21 (RIN2); no longer U4.23 (RIN1)
- net CV1_ADC: now also U1.39 (IO1); no longer U1.17 (IO9)
- net CV2_ADC: now also U1.38 (IO2); no longer U1.18 (IO10)
Other:
- note added: "AUDIO IN L/R: 100k / 22k (x0.18) -> U7C/U7D follower -> 1u -> 1k -> LIN2/RIN2 (100k to VMID). +/-5 V -> +/-0.9 V; codec PGA sets the gain. No IN R normal: firmware handles mono."
- note added: "CV IN 1/2: tip normalled to +5V -> RV1/RV2 50k attenuator -> U7B/U7A TL074 follower -> 100k / 56k to +3V3 / 120k to GND, BAT54SW clamp, 1n -> U6B/U6A MCP6002 follower -> IO1/IO2. Unpatched: RV = 0..+5 V knob. Patched: RV scales the CV. -5.9..+6.0 V -> 0..3.3 V."
- note added: "ES8388 CODEC (Bread Modular U4): I2S IO11-14/IO21 through 33R, I2C IO38 (CCLK) / IO39 (CDATA), CE = GND (0x10). Inputs on LIN2/RIN2. +3V3 -> R5 10R -> +3V3_8388."
- note removed: "AUDIO IN L/R: 100k / 22k (x0.18) -> U7C/U7D follower -> 1u -> 1k -> LIN1/RIN1 (100k to VMID). +/-5 V -> +/-0.9 V; codec PGA sets the gain. No IN R normal: firmware handles mono."
- note removed: "CV IN 1/2: tip normalled to +5V -> RV1/RV2 50k attenuator -> U7B/U7A TL074 follower -> 100k / 56k to +3V3 / 120k to GND, BAT54SW clamp, 1n -> U6B/U6A MCP6002 follower -> IO9/IO10. Unpatched: RV = 0..+5 V knob. Patched: RV scales the CV. -5.9..+6.0 V -> 0..3.3 V."
- note removed: "ES8388 CODEC (Bread Modular U4): I2S IO11-14/IO21 through 33R, I2C IO47 (CCLK) / IO48 (CDATA), CE = GND (0x10). +3V3 -> R5 10R -> +3V3_8388."
Changed lines of the file:
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@@
 		)
 	)
-	(text "AUDIO IN L/R: 100k / 22k (x0.18) -> U7C/U7D follower -> 1u -> 1k -> LIN1/RIN1 (100k to VMID).\n+/-5 V -> +/-0.9 V; codec PGA sets the gain. No IN R normal: firmware handles mono."
+	(text "AUDIO IN L/R: 100k / 22k (x0.18) -> U7C/U7D follower -> 1u -> 1k -> LIN2/RIN2 (100k to VMID).\n+/-5 V -> +/-0.9 V; codec PGA sets the gain. No IN R normal: firmware handles mono."
 		(exclude_from_sim no)
 		(at 436.88 33.02 0)
@@
 		)
 	)
-	(text "CV IN 1/2: tip normalled to +5V -> RV1/RV2 50k attenuator -> U7B/U7A TL074 follower\n-> 100k / 56k to +3V3 / 120k to GND, BAT54SW clamp, 1n -> U6B/U6A MCP6002 follower -> IO9/IO10.\nUnpatched: RV = 0..+5 V knob. Patched: RV scales the CV. -5.9..+6.0 V -> 0..3.3 V."
+	(text "CV IN 1/2: tip normalled to +5V -> RV1/RV2 50k attenuator -> U7B/U7A TL074 follower\n-> 100k / 56k to +3V3 / 120k to GND, BAT54SW clamp, 1n -> U6B/U6A MCP6002 follower -> IO1/IO2.\nUnpatched: RV = 0..+5 V knob. Patched: RV scales the CV. -5.9..+6.0 V -> 0..3.3 V."
 		(exclude_from_sim no)
 		(at 20.32 203.2 0)
@@
 		)
 	)
-	(text "ES8388 CODEC (Bread Modular U4): I2S IO11-14/IO21 through 33R,\nI2C IO47 (CCLK) / IO48 (CDATA), CE = GND (0x10). +3V3 -> R5 10R -> +3V3_8388."
+	(text "ES8388 CODEC (Bread Modular U4): I2S IO11-14/IO21 through 33R,\nI2C IO38 (CCLK) / IO39 (CDATA), CE = GND (0x10). Inputs on LIN2/RIN2. +3V3 -> R5 10R -> +3V3_8388."
 		(exclude_from_sim no)
 		(at 330.2 71.12 0)
@@
 	)
 	(no_connect
-		(at 294.64 157.48)
-	)
-	(no_connect
-		(at 406.4 110.49)
+		(at 264.16 157.48)
 	)
 	(no_connect
@@
 	)
 	(no_connect
+		(at 406.4 114.3)
+	)
+	(no_connect
+		(at 294.64 172.72)
+	)
+	(no_connect
 		(at 264.16 172.72)
 	)
@@
 	)
 	(no_connect
-		(at 406.4 106.68)
+		(at 264.16 160.02)
 	)
 	(no_connect
@@
 	)
 	(no_connect
-		(at 264.16 139.7)
-	)
-	(no_connect
 		(at 264.16 175.26)
 	)
@@
 	)
 	(no_connect
-		(at 264.16 137.16)
+		(at 294.64 165.1)
 	)
 	(no_connect
-		(at 294.64 165.1)
+		(at 294.64 175.26)
+	)
+	(no_connect
+		(at 406.4 118.11)
 	)
 	(no_connect
@@
 	)
 	(no_connect
-		(at 294.64 154.94)
-	)
-	(no_connect
 		(at 449.58 53.34)
 	)
@@
 	(wire
 		(pts
-			(xy 261.62 160.02) (xy 264.16 160.02)
-		)
-		(stroke
-			(width 0)
-			(type default)
-		)
-	)
-	(wire
-		(pts
 			(xy 520.7 116.84) (xy 520.7 119.38)
 		)
@@
 	(wire
 		(pts
-			(xy 406.4 118.11) (xy 408.94 118.11)
+			(xy 261.62 137.16) (xy 264.16 137.16)
 		)
 		(stroke
@@
 	(wire
 		(pts
-			(xy 421.64 153.67) (xy 421.64 156.21)
+			(xy 406.4 106.68) (xy 408.94 106.68)
 		)
 		(stroke
@@
 	(wire
 		(pts
-			(xy 374.65 95.25) (xy 377.19 95.25)
+			(xy 421.64 153.67) (xy 421.64 156.21)
 		)
 		(stroke
@@
 	(wire
 		(pts
-			(xy 27.94 226.06) (xy 30.48 226.06)
+			(xy 374.65 95.25) (xy 377.19 95.25)
 		)
 		(stroke
@@
 	(wire
 		(pts
-			(xy 528.32 200.66) (xy 533.4 200.66)
+			(xy 27.94 226.06) (xy 30.48 226.06)
 		)
 		(stroke
@@
 	(wire
 		(pts
-			(xy 76.2 142.24) (xy 80.01 142.24)
+			(xy 528.32 200.66) (xy 533.4 200.66)
 		)
 		(stroke
@@
 	(wire
 		(pts
-			(xy 421.64 184.15) (xy 421.64 186.69)
+			(xy 76.2 142.24) (xy 80.01 142.24)
 		)
 		(stroke
@@
 	(wire
 		(pts
-			(xy 71.12 229.87) (xy 71.12 236.22)
+			(xy 421.64 184.15) (xy 421.64 186.69)
 		)
 		(stroke
@@
 	(wire
 		(pts
-			(xy 294.64 172.72) (xy 297.18 172.72)
+			(xy 71.12 229.87) (xy 71.12 236.22)
 		)
 		(stroke
@@
 	(wire
 		(pts
+			(xy 261.62 139.7) (xy 264.16 139.7)
+		)
+		(stroke
+			(width 0)
+			(type default)
+		)
+	)
+	(wire
+		(pts
 			(xy 474.98 86.36) (xy 495.3 86.36)
 		)
@@
 	(wire
 		(pts
-			(xy 261.62 157.48) (xy 264.16 157.48)
-		)
-		(stroke
-			(width 0)
-			(type default)
-		)
-	)
-	(wire
-		(pts
 			(xy 99.06 287.02) (xy 104.14 287.02)
 		)
@@
 	(wire
 		(pts
+			(xy 294.64 157.48) (xy 297.18 157.48)
+		)
+		(stroke
+			(width 0)
+			(type default)
+		)
+	)
+	(wire
+		(pts
 			(xy 30.48 154.94) (xy 30.48 157.48)
 		)
@@
 	(wire
 		(pts
-			(xy 243.84 129.54) (xy 256.54 129.54)
+			(xy 406.4 110.49) (xy 408.94 110.49)
 		)
 		(stroke
@@
 	(wire
 		(pts
-			(xy 261.62 106.68) (xy 264.16 106.68)
+			(xy 243.84 129.54) (xy 256.54 129.54)
 		)
 		(stroke
@@
 	(wire
 		(pts
-			(xy 441.96 184.15) (xy 441.96 186.69)
+			(xy 261.62 106.68) (xy 264.16 106.68)
 		)
 		(stroke
@@
 	(wire
 		(pts
-			(xy 50.8 232.41) (xy 53.34 232.41)
+			(xy 441.96 184.15) (xy 441.96 186.69)
 		)
 		(stroke
@@
 	(wire
 		(pts
-			(xy 289.56 116.84) (xy 299.72 116.84)
+			(xy 50.8 232.41) (xy 53.34 232.41)
 		)
 		(stroke
@@
 	(wire
 		(pts
-			(xy 520.7 152.4) (xy 523.24 152.4)
+			(xy 289.56 116.84) (xy 299.72 116.84)
 		)
 		(stroke
@@
 	(wire
 		(pts
-			(xy 294.64 132.08) (xy 297.18 132.08)
+			(xy 520.7 152.4) (xy 523.24 152.4)
 		)
 		(stroke
@@
 	(wire
 		(pts
-			(xy 406.4 95.25) (xy 408.94 95.25)
+			(xy 294.64 132.08) (xy 297.18 132.08)
 		)
 		(stroke
@@
 	(wire
 		(pts
-			(xy 294.64 175.26) (xy 297.18 175.26)
+			(xy 406.4 95.25) (xy 408.94 95.25)
 		)
 		(stroke
@@
 	(wire
 		(pts
+			(xy 294.64 154.94) (xy 297.18 154.94)
+		)
+		(stroke
+			(width 0)
+			(type default)
+		)
+	)
+	(wire
+		(pts
 			(xy 99.06 276.86) (xy 99.06 279.4)
 		)
@@
 	(wire
 		(pts
-			(xy 406.4 114.3) (xy 408.94 114.3)
-		)
-		(stroke
-			(width 0)
-			(type default)
-		)
-	)
-	(wire
-		(pts
 			(xy 45.72 231.14) (xy 45.72 233.68)
 		)
@@
 		)
 	)
-	(label "CV1_ADC"
-		(at 261.62 157.48 180)
+	(label "CV2_ADC"
+		(at 261.62 139.7 180)
 		(effects
 			(font
@@
 	)
 	(label "CODEC_LIN"
-		(at 408.94 118.11 0)
+		(at 408.94 110.49 0)
 		(effects
 			(font
@@
 		)
 	)
-	(label "CV2_ADC"
-		(at 261.62 160.02 180)
+	(label "BUTTON"
+		(at 261.62 154.94 180)
 		(effects
 			(font
@@
 	)
 	(label "CODEC_RIN"
-		(at 408.94 114.3 0)
+		(at 408.94 106.68 0)
 		(effects
 			(font
@@
 	)
 	(label "CDATA"
-		(at 297.18 175.26 0)
+		(at 297.18 157.48 0)
 		(effects
 			(font
@@
 		)
 	)
-	(label "BUTTON"
-		(at 261.62 154.94 180)
+	(label "CV1_ADC"
+		(at 261.62 137.16 180)
 		(effects
 			(font
@@
 	)
 	(label "CCLK"
-		(at 297.18 172.72 0)
+		(at 297.18 154.94 0)
 		(effects
 			(font
@@
 			)
 		)
-		(property "Note" "I2C CCLK pull-up (Bread Modular R25)"
+		(property "Note" "I2C CCLK pull-up to +3V3 (Bread Modular R25: +3V3_8388; R1 layout uses the +3V3 plane, same level through the 10R)"
 			(at 452.12 190.5 0)
 			(hide yes)
@@
 			)
 		)
-		(property "Value" "+3V3_8388"
+		(property "Value" "+3V3"
 			(at 441.96 180.34 0)
 			(show_name no)
@@
 			)
 		)
-		(property "Note" "I2C CDATA pull-up (Bread Modular R24)"
+		(property "Note" "I2C CDATA pull-up to +3V3 (Bread Modular R24: +3V3_8388; R1 layout uses the +3V3 plane, same level through the 10R)"
 			(at 441.96 190.5 0)
 			(hide yes)
@@
 			)
 		)
-		(property "Footprint" "32BIT:R_0603_1608Metric"
+		(property "Footprint" "32BIT:R_0402_1005Metric"
 			(at 523.24 57.15 0)
 			(hide yes)
@@
 			)
 		)
-		(property "Note" "Input bias to VMID (Bread Modular R19/R16)"
+		(property "Note" "Input bias to VMID (Bread Modular R19/R16); 0402 to fit beside the codec (R1)"
 			(at 523.24 57.15 0)
 			(hide yes)
@@
 			)
 		)
-		(property "LCSC" "C25803"
+		(property "LCSC" "C25741"
 			(at 523.24 57.15 0)
 			(hide yes)
@@
 			)
 		)
-		(property "MPN" "0603WAF1003T5E"
+		(property "MPN" "0402WGF1003TCE"
 			(at 523.24 57.15 0)
 			(hide yes)
@@
 			)
 		)
-		(property "Footprint" "32BIT:R_0603_1608Metric"
+		(property "Footprint" "32BIT:R_0402_1005Metric"
 			(at 523.24 82.55 0)
 			(hide yes)
@@
 			)
 		)
-		(property "Note" "Input bias to VMID (Bread Modular R19/R16)"
+		(property "Note" "Input bias to VMID (Bread Modular R19/R16); 0402 to fit beside the codec (R1)"
 			(at 523.24 82.55 0)
 			(hide yes)
@@
 			)
 		)
-		(property "LCSC" "C25803"
+		(property "LCSC" "C25741"
 			(at 523.24 82.55 0)
 			(hide yes)
@@
 			)
 		)
-		(property "MPN" "0603WAF1003T5E"
+		(property "MPN" "0402WGF1003TCE"
 			(at 523.24 82.55 0)
 			(hide yes)
