File: modules/usb-audio/hardware/usb-audio.kicad_pcb (KiCad board)
At the start: 4 copper layers, 29 x 110 mm, 81 parts, among them J1 Eurorack_2x5, J2 PJ301M-12, J3 PJ301M-12, J4 PJ301M-12, J5 PJ301M-12, J6 MCU_L, J7 MCU_R, J8 SWD, SW1 RESET, SW2 BOOT, U1 AMS1117-5.0, U2 AMS1117-3.3, U3 CS4270, U4 OPA1679, U5 OPA1678, U6 OPA1679, Y1 24.576MHz

Commit message: Add USB-Audio module.
Parts:
- added C31: 100n, USBAUDIO:C_0603_1608Metric, B.Cu at (111.9, 140.4)
- added C32: 100n, USBAUDIO:C_0603_1608Metric, B.Cu at (118.0, 131.7)
- added U7: OPA1678, USBAUDIO:SOIC-8_3.9x4.9mm_P1.27mm, B.Cu at (116.0, 137.0)
- U4: value OPA1679 -> OPA1678; footprint USBAUDIO:SOIC-14_3.9x8.7mm_P1.27mm -> USBAUDIO:SOIC-8_3.9x4.9mm_P1.27mm
- moved R31 42.9 mm to (110.6, 76.0), turned to -90 degrees
- moved C22 39.6 mm to (106.0, 76.8), turned to 180 degrees
- moved R30 36.2 mm to (108.9, 76.8), turned to -90 degrees
- moved C23 31.1 mm to (112.5, 80.3), turned to -90 degrees
- moved R21 28.3 mm to (122.0, 114.4), turned to 90 degrees
- moved C24 27.5 mm to (126.5, 107.7)
- moved R34 27.5 mm to (106.2, 84.7), turned to 180 degrees
- moved R42 27.1 mm to (112.6, 97.1), turned to -90 degrees
- moved C28 26.9 mm to (112.5, 83.5), turned to -90 degrees
- moved R32 24.4 mm to (106.2, 86.4), turned to 0 degrees
- moved U5 23.8 mm to (108.0, 81.1), turned to 0 degrees
- moved C29 23.2 mm to (112.5, 86.6)
- moved C26 22.7 mm to (113.2, 107.7)
- moved R43 22.3 mm to (112.6, 93.9), turned to 90 degrees
- moved R40 18.5 mm to (122.0, 94.4), turned to -90 degrees
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Connections:
- R36 pad 1: Net-(U4C--) -> Net-(U7A--)
- R37 pad 1: Net-(U4D--) -> Net-(U7B--)
- RV3 pad 2: Net-(U4C-+) -> Net-(U7A-+)
- RV4 pad 2: Net-(U4D-+) -> Net-(U7B-+)
- U4 pad 4: +12V_F -> -12V_F
- U4 pad 8: Net-(U4C--) -> +12V_F
Routing:
- net Net-(U4D-+): track 78.2 -> 0.00 mm, vias 2 -> 0
- net Net-(U4D--): track 73.3 -> 0.00 mm, vias 2 -> 0
- net Net-(U4C-+): track 56.8 -> 0.00 mm, vias 2 -> 0
- net /VREF_OUT: track 75.1 -> 20.4 mm, vias 5 -> 0
- net /DAC_B: track 57.0 -> 2.31 mm, vias 2 -> 0
- net Net-(U4C--): track 51.5 -> 0.00 mm, vias 2 -> 0
- net +5VA: track 126.5 -> 81.7 mm, vias 4 -> 5
- net /DAC_A: track 50.8 -> 7.78 mm, vias 2 -> 0
- net Net-(R21-Pad1): track 39.3 -> 4.28 mm, vias 2 -> 0
- net /VB_IN: track 12.7 -> 38.4 mm, vias 0 -> 2
- net /IN1: track 62.8 -> 38.4 mm, vias 2 -> 1
- net Net-(U7B-+): track 0.00 -> 22.6 mm
- net +3V3_C: track 22.0 -> 44.4 mm, vias 0 -> 3
- net Net-(U7A--): track 0.00 -> 19.1 mm
- net /I2S_ADC: track 2.46 -> 21.3 mm, vias 0 -> 1
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- added copper zone on In2.Cu, net +5VA

Commit message: Improve the USB Out module.
Parts:
- added R38: 2k, USBAUDIO:R_1206_3216Metric, B.Cu at (127.3, 129.0)
- added R39: 2k, USBAUDIO:R_1206_3216Metric, B.Cu at (127.3, 145.0)
- R36, R37: value 1k -> 2k
Routing:
- net /OUT2: track 5.92 -> 16.8 mm, vias 0 -> 2
- net /OUT1: track 5.92 -> 16.8 mm, vias 0 -> 2
- net Net-(U7B--): track 16.8 -> 18.9 mm
- net Net-(U7A--): track 19.1 -> 21.1 mm
