File: modules/acid/panels/front-pcb/acid-panel.kicad_pcb (KiCad board)
At the start: 2 copper layers, 40.3 x 128.5 mm, 24 parts

Commit message: Move panel holes similar to MIDI.
Parts:
- moved H1 5.08 mm to (112.6, 53.0)
- moved H3 5.08 mm to (112.6, 175.5)
Changed lines of the file:
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@@
 	(footprint ""
 		(layer "F.Cu")
-		(at 107.5 53)
+		(at 112.58 53)
 		(property "Reference" "H1"
 			(at 0 0 0)
@@
 	(footprint ""
 		(layer "F.Cu")
-		(at 107.5 175.5)
+		(at 112.58 175.5)
 		(property "Reference" "H3"
 			(at 0 0 0)
