File: modules/hats/panels/front-pcb/hats-panel.kicad_pcb (KiCad board)
At the start: 2 copper layers, 30 x 128.5 mm, 13 parts

Commit message: Improve the hats module.
Parts:
- removed H12, H13: MECHANICAL_NPTH, 
- moved H10 10.0 mm to (122.2, 125.0)
- moved H9 10.0 mm to (107.8, 125.0)
Other:
- board text removed: "REC"

Commit message: Change the CV light position.
Parts:
- moved H11 39.8 mm to (126.0, 143.0)

Commit message: Move panel holes similar to MIDI.
Parts:
- moved H1 5.08 mm to (112.6, 53.0)
- moved H2 5.08 mm to (112.6, 175.5)
Changed lines of the file:
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@@
 	(footprint ""
 		(layer "F.Cu")
-		(at 107.5 175.5)
+		(at 112.58 175.5)
 		(property "Reference" "H2"
 			(at 0 0 0)
@@
 	(footprint ""
 		(layer "F.Cu")
-		(at 107.5 53)
+		(at 112.58 53)
 		(property "Reference" "H1"
 			(at 0 0 0)
