File: modules/line-in/hardware/line-in.kicad_pcb (KiCad board)
At the start: 2 copper layers, 19 x 110 mm, 37 parts, among them J1 PJ366ST, J10 Eurorack_2x5, J2 PJ301M-12, J3 PJ301M-12, J4 PJ301M-12, U1 TL072CDT, U2 TL072CDT, U3 TL072CDT

Commit message: Added LINE In Protections.
Parts:
- added D3: BAV199, LineIn:SOT-23, B.Cu at (110.0, 85.0)
- added D4: BAV199, LineIn:SOT-23, B.Cu at (110.0, 89.0)
- added D5: BAV199, LineIn:SOT-23, B.Cu at (110.0, 107.0)
- added D6: BAV199, LineIn:SOT-23, B.Cu at (110.0, 110.9)
- added R13: 10k, LineIn:R_0603_1608Metric, B.Cu at (102.5, 96.8)
- added R14: 10k, LineIn:R_0603_1608Metric, B.Cu at (102.5, 118.0)
Connections:
- C10 pad 2: /AC_R -> /COUP_R
- C9 pad 2: /AC_L -> /COUP_L
- R1 pad 1: /AC_L -> /COUP_L
- R2 pad 1: /AC_R -> /COUP_R
Routing:
- net /AC_L: track 5.56 -> 30.3 mm, vias 0 -> 3
- net /AC_R: track 5.56 -> 29.3 mm, vias 0 -> 3
- net /COUP_R: track 0.00 -> 7.19 mm, vias 0 -> 2
- net /COUP_L: track 0.00 -> 7.19 mm, vias 0 -> 2
- net GND: track 21.9 -> 25.2 mm, vias 14 -> 17
Other:
- board text added: "LINE IN R2"
- board text removed: "LINE IN R1"
