File: modules/env/hardware/env.kicad_pcb (KiCad board)
At the start: 2 copper layers, 29 x 110 mm, 52 parts, among them J1 PJ301M-12, J2 PJ301M-12, J3 Eurorack_2x5, J4 UPDI, J5 PJ301M-12, J6 PJ301M-12, Q1 MMBT3904, Q2 MMBT3904, SW1 MODE, SW2 REC, U1 HT7533-1, U2 ATtiny1616-MNR, U3 TL072

Commit message: Run the env module MCU at 5V.
Parts:
- R5, R6, R7, R8: value 330 -> 1k
- U1: value HT7533-1 -> HT7550-1
Connections:
- net +3V3 renamed +5V
