File: modules/low/hardware/low.kicad_pcb (KiCad board)
At the start: 2 copper layers, 29 x 110 mm, 70 parts, among them J1 PJ301M-12, J10 Eurorack_2x5, J11 UPDI, J2 PJ301M-12, J3 PJ301M-12, J4 PJ301M-12, Q1 MMBT3904, U1 HT7533-1, U2 ATtiny1616-MNR, U3 MCP6002, U4 TS5A23157, U5 VTL5C, U6 MCP6002, U7 VTL5C, U8 MCP6002, U9 TL072

Commit message: Make sure LOW module is FAB ready.
Parts:
- moved C16 0.50 mm to (121.3, 167.4)
- moved U5 0.50 mm to (109.5, 133.3)
- moved U9 0.45 mm to (122.4, 162.9)
- moved J11 0.30 mm to (126.7, 80.0)
- moved C5 0.20 mm to (103.2, 142.7)
- moved D4 0.20 mm to (127.2, 116.3)
- moved C12 0.10 mm to (127.0, 139.6)
Routing:
- net +3V3: track 268.1 -> 264.0 mm
- net /DETUNE: track 20.9 -> 22.0 mm
- net +12V_F: track 40.9 -> 40.1 mm
- net /VMID_LPG: track 19.4 -> 18.6 mm
- net /LPF1: track 26.5 -> 26.0 mm
- net /VAC_POS: track 21.8 -> 22.3 mm
- net GND: track 39.6 -> 39.5 mm, vias 22 -> 23

Commit message: Add LOW module firmware. Also make sure MIDI P/D works fine.
Other:
- board text added: "D"
- board text added: "P"
- board text removed: "PROT RX DIR"
Changed lines of the file:
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@@
 		)
 	)
-	(gr_text "PROT RX DIR"
-		(at 110.4 81.95 0)
+	(gr_text "P"
+		(at 109.1 82 0)
 		(layer "B.SilkS")
 		(effects
 			(font
-				(size 0.8 0.8)
+				(size 1 1)
 				(thickness 0.15)
 			)
+			(justify mirror)
+		)
+	)
+	(gr_text "D"
+		(at 111.7 82 0)
+		(layer "B.SilkS")
+		(effects
+			(font
+				(size 1 1)
+				(thickness 0.15)
+			)
