File: modules/hats/hardware/hats.kicad_pcb (KiCad board)
At the start: 4 copper layers, 29 x 110 mm, 104 parts, among them J1 PJ301M-12, J10 Eurorack_2x5, J11 UPDI_NOISE, J12 UPDI_HIHAT, J2 PJ301M-12, J3 PJ301M-12, J4 PJ301M-12, Q1 MMBT3904, Q2 SS8050, Q3 SS8550, Q4 SS8050, SW1 REC, U1 HT7533-1, U10 TL072, U2 ATtiny1616-MNR, U3 ATtiny1616-MNR, U4 MCP6002, U5 TS5A23157, U6 MCP6002, U7 VTL5C, U8 MCP6002, U9 MCP6002

Commit message: Improve the hats module.
Parts:
- removed D6: LED_3mm_red, HATS:LED_D3.0mm
- removed R48: 330, HATS:R_0603_1608Metric
- removed SW1: REC, HATS:SW_PUSH_6mm_H7.3mm
- added D7: BAV199, HATS:SOT-23, B.Cu at (117.0, 79.0)
- added R49: 22k, HATS:R_0603_1608Metric, B.Cu at (119.0, 70.5)
- R14: value 1M -> 470k
- moved RV3 8.99 mm to (107.6, 124.5), turned to 180 degrees
- moved RV4 8.99 mm to (122.1, 124.5), turned to 180 degrees
- moved R23 8.29 mm to (122.3, 134.6)
- moved Q3 6.50 mm to (122.2, 122.5)
- moved R21 5.75 mm to (122.1, 132.7)
- moved R36 5.46 mm to (122.2, 113.8)
- moved D4 4.30 mm to (115.0, 120.7), turned to 0 degrees
- moved R27 4.30 mm to (106.5, 121.6)
- moved U7 3.30 mm to (107.0, 138.0)
- moved Q2 3.20 mm to (115.0, 117.3)
- moved R19 3.14 mm to (117.1, 129.4)
- moved R25 3.11 mm to (109.3, 113.6), turned to 0 degrees
- moved R24 1.60 mm to (106.2, 113.6), turned to 0 degrees
- moved Q4 1.25 mm to (125.2, 129.2), turned to 0 degrees
- moved R18 1.20 mm to (114.0, 129.4)
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Connections:
- J2 pad TN: /NIN_SENSE -> /NIN_SENSE_RAW
- U2 pad 17: /REC_SW -> unconnected-(U2-PC2-Pad17)
- U3 pad 17: /REC_SW -> unconnected-(U3-PC2-Pad17)
- U3 pad 18: /LED_REC -> unconnected-(U3-PC3-Pad18)
Routing:
- net /REC_SW: track 83.2 -> 0.00 mm, vias 3 -> 0
- net /LED_REC: track 70.9 -> 0.00 mm, vias 4 -> 0
- net /VCA_IN: track 22.4 -> 35.4 mm, vias 0 -> 4
- net /VMID_H: track 78.1 -> 66.5 mm, vias 7 -> 8
- net /NIN_SENSE: track 11.0 -> 22.4 mm, vias 0 -> 2
- net /VAC_K: track 14.7 -> 25.1 mm, vias 0 -> 2
- net GND: track 63.2 -> 54.3 mm
- net /TRIG: track 11.1 -> 19.5 mm
- net /HH_IN: track 78.9 -> 87.1 mm, vias 2 -> 4
- net /GATE_OPEN: track 2.64 -> 9.98 mm
- net /VCA_FB: track 5.27 -> 12.2 mm, vias 0 -> 2
- net /DECAY_R: track 4.12 -> 10.6 mm
- net /NIN_SENSE_RAW: track 0.00 -> 5.95 mm
- net /ENV_CAP: track 15.1 -> 21.0 mm, vias 2 -> 0
- net /ENV_BUF: track 37.2 -> 42.9 mm
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Other:
- board text added: "HATS R2"
- board text removed: "HATS P3"

Commit message: Change the CV light position.
Parts:
- moved R47 40.6 mm to (121.8, 142.6)
- moved D5 40.5 mm to (127.3, 143.0), turned to 180 degrees
Routing:
- net /CVO_AMP: track 70.8 -> 21.7 mm, vias 2 -> 0
Changed lines of the file:
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@@
 	(footprint "HATS:LED_D3.0mm"
 		(layer "F.Cu")
-		(at 113.73 104.8)
+		(at 127.27 143 180)
 		(descr "LED, diameter 3.0mm, 2 pins, generated by kicad-footprint-generator")
 		(tags "LED")
 		(property "Reference" "D5"
-			(at 1.27 -2.96 0)
+			(at 1.27 -2.96 180)
 			(layer "F.Fab")
 			(effects
@@
 		)
 		(property "Value" "LED_3mm_red"
-			(at 1.27 2.96 0)
+			(at 1.27 2.96 180)
 			(layer "F.Fab")
 			(hide yes)
@@
 		)
 		(property "Datasheet" ""
-			(at 0 0 0)
+			(at 0 0 180)
 			(layer "F.Fab")
 			(hide yes)
@@
 		)
 		(property "Description" "Light emitting diode"
-			(at 0 0 0)
+			(at 0 0 180)
 			(layer "F.Fab")
 			(hide yes)
@@
 		)
 		(property "KiLib_Generator" "LED/THT"
-			(at 0 0 0)
+			(at 0 0 180)
 			(layer "F.SilkS")
 			(hide yes)
@@
 		)
 		(property "Note" "HAT CV LED (follows the envelope). Hand-soldered 3 mm THT, dome flush with the panel (as modules/8bit)"
-			(at 0 0 0)
+			(at 0 0 180)
 			(layer "F.SilkS")
 			(hide yes)
@@
 		(duplicate_pad_numbers_are_jumpers no)
 		(fp_line
-			(start -0.29 -1.236)
-			(end -0.29 -1.08)
+			(start -0.29 1.08)
+			(end -0.29 1.236)
 			(stroke
 				(width 0.12)
@@
 		)
 		(fp_line
-			(start -0.29 1.08)
-			(end -0.29 1.236)
+			(start -0.29 -1.236)
+			(end -0.29 -1.08)
 			(stroke
 				(width 0.12)
@@
 		)
 		(fp_arc
-			(start -0.29 -1.235516)
-			(mid 1.36566 -1.987699)
-			(end 2.941437 -1.08)
+			(start 2.941437 1.08)
+			(mid 1.36566 1.987699)
+			(end -0.29 1.235516)
 			(stroke
 				(width 0.12)
@@
 		)
 		(fp_arc
-			(start 0.229039 -1.08)
-			(mid 1.27 -1.5)
-			(end 2.310961 -1.08)
+			(start 2.310961 1.08)
+			(mid 1.27 1.5)
+			(end 0.229039 1.08)
 			(stroke
 				(width 0.12)
@@
 		)
 		(fp_arc
-			(start 2.310961 1.08)
-			(mid 1.27 1.5)
-			(end 0.229039 1.08)
+			(start 0.229039 -1.08)
+			(mid 1.27 -1.5)
+			(end 2.310961 -1.08)
 			(stroke
 				(width 0.12)
@@
 		)
 		(fp_arc
-			(start 2.941437 1.08)
-			(mid 1.36566 1.987699)
-			(end -0.29 1.235516)
+			(start -0.29 -1.235516)
+			(mid 1.36566 -1.987699)
+			(end 2.941437 -1.08)
 			(stroke
 				(width 0.12)
@@
 		)
 		(fp_text user "${REFERENCE}"
-			(at 1.27 0 0)
+			(at 1.27 0 180)
 			(layer "F.Fab")
 			(effects
@@
 		)
 		(point
-			(at 115 104.8)
+			(at 126 143)
 			(size 2)
 			(layer "F.Fab")
 		)
 		(pad "1" thru_hole rect
-			(at 0 0)
+			(at 0 0 180)
 			(size 1.8 1.8)
 			(drill 0.9)
@@
 		)
 		(pad "2" thru_hole circle
-			(at 2.54 0)
+			(at 2.54 0 180)
 			(size 1.8 1.8)
 			(drill 0.9)
@@
 	(footprint "HATS:R_0603_1608Metric"
 		(layer "B.Cu")
-		(at 114.9 102.6)
+		(at 121.825 142.6)
 		(descr "Resistor SMD 0603 (1608 Metric), square (rectangular) end terminal, IPC-7351 nominal, (Body size source: IPC-SM-782 page 72, https://www.pcb-3d.com/wordpress/wp-content/uploads/ipc-sm-782a_amendment_1_and_2.pdf)")
 		(tags "resistor")
@@
 	)
 	(segment
-		(start 115.725 102.6)
-		(end 115.725 104.255)
+		(start 123.05 143)
+		(end 124.73 143)
 		(width 0.25)
 		(layer "B.Cu")
@@
 	)
 	(segment
-		(start 115.725 104.255)
-		(end 116.27 104.8)
+		(start 122.65 142.6)
+		(end 123.05 143)
 		(width 0.25)
 		(layer "B.Cu")
@@
 	)
 	(segment
-		(start 117.15 109.1)
-		(end 120.5 112.45)
-		(width 0.2)
-		(layer "F.Cu")
-		(net "/CVO_AMP")
-	)
-	(segment
-		(start 123.5 115.05)
-		(end 123.5 126.1)
-		(width 0.2)
-		(layer "F.Cu")
-		(net "/CVO_AMP")
-	)
-	(segment
-		(start 120.5 112.45)
-		(end 120.9 112.45)
-		(width 0.2)
-		(layer "F.Cu")
-		(net "/CVO_AMP")
-	)
-	(segment
-		(start 123.5 126.1)
-		(end 126.65 129.25)
-		(width 0.2)
-		(layer "F.Cu")
-		(net "/CVO_AMP")
-	)
-	(segment
-		(start 127.35 138)
-		(end 127.35 138.5)
-		(width 0.25)
-		(layer "F.Cu")
-		(net "/CVO_AMP")
-	)
-	(segment
-		(start 127.35 138.5)
-		(end 119.25 146.6)
-		(width 0.25)
-		(layer "F.Cu")
-		(net "/CVO_AMP")
-	)
-	(segment
-		(start 120.9 112.45)
-		(end 123.5 115.05)
-		(width 0.2)
-		(layer "F.Cu")
-		(net "/CVO_AMP")
-	)
-	(segment
-		(start 115.9 109.1)
-		(end 117.15 109.1)
-		(width 0.2)
-		(layer "F.Cu")
-		(net "/CVO_AMP")
-	)
-	(segment
-		(start 126.65 137.3)
-		(end 127.35 138)
-		(width 0.25)
-		(layer "F.Cu")
-		(net "/CVO_AMP")
-	)
-	(segment
-		(start 115 108.2)
-		(end 115.9 109.1)
-		(width 0.2)
-		(layer "F.Cu")
-		(net "/CVO_AMP")
-	)
-	(segment
-		(start 115 103.5)
-		(end 115 108.2)
-		(width 0.25)
-		(layer "F.Cu")
-		(net "/CVO_AMP")
-	)
-	(segment
-		(start 126.65 129.25)
-		(end 126.65 137.3)
-		(width 0.2)
-		(layer "F.Cu")
-		(net "/CVO_AMP")
-	)
-	(via
-		(at 115 103.5)
-		(size 0.6)
-		(drill 0.3)
-		(layers "F.Cu" "B.Cu")
-		(net "/CVO_AMP")
-	)
-	(via
-		(at 119.25 146.6)
-		(size 0.6)
-		(drill 0.3)
-		(layers "F.Cu" "B.Cu")
-		(net "/CVO_AMP")
-	)
-	(segment
 		(start 126.75 150.3625)
 		(end 127.15 149.9625)
@@
 	)
 	(segment
+		(start 121 143)
+		(end 119.25 144.75)
+		(width 0.25)
+		(layer "B.Cu")
+		(net "/CVO_AMP")
+	)
+	(segment
 		(start 118.8 149.75)
 		(end 118.8 146.625)
@@
 	)
 	(segment
-		(start 114.075 102.6)
-		(end 115 103.5)
+		(start 121 142.6)
+		(end 121 143)
+		(width 0.25)
+		(layer "B.Cu")
+		(net "/CVO_AMP")
+	)
+	(segment
+		(start 119.25 144.75)
+		(end 119.25 146.6)
 		(width 0.25)
 		(layer "B.Cu")

Commit message: Add standard UPDI labels for 32bit to hats.
Other:
- board text added: "D"
- board text added: "P"
Changed lines of the file:
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@@
 	)
 	(embedded_fonts no)
+	(gr_text "P"
+		(at 116.25 67.6 0)
+		(layer "B.SilkS")
+		(effects
+			(font
+				(size 1 1)
+				(thickness 0.15)
+			)
+			(justify mirror)
+		)
+	)
+	(gr_text "D"
+		(at 113.65 67.6 0)
+		(layer "B.SilkS")
+		(effects
+			(font
+				(size 1 1)
+				(thickness 0.15)
+			)
+			(justify mirror)
+		)
+	)
 )
