File: modules/usb-power-45w/hardware/usb-power-45w.kicad_sch (KiCad schematic)
At the start: 80 parts, among them J1 TYPE-C-31-M-12, J2 IDC 2x8 box header, J3 IDC 2x8 box header, Q1 MMBT3906, SW1 TL3340AF160QG, U1 CH224A, U2 TPS62933FDRLR, U3 TPS62933FDRLR, U4 LMR38020FDDAR, U5 TPS259470ARPWR

Commit message: Revise USB power input protection and board-side current limit
Replace the low-voltage eFuse with TPS16630, coordinate input and PD-controller protection, and set a 4.186 A nominal board-side limit. Upgrade the reverse-blocking diode while preserving all three converter stages.

Include sourcing evidence, S4/S5 design records, native schematic/BOM/PDF updates and electrical parity checks. Schematic only: thermal, fault, supplier-document and assembly-policy gates remain open.
Parts:
- removed C4: 10n, USBPOWER45:C_0603_1608Metric, symbol USBPOWER45:C
- added D10: SS1060, USBPOWER45:D_SMC, symbol USBPOWER45:D_Schottky
- added D11: SS34, USBPOWER45:D_SMA, symbol USBPOWER45:D_Schottky
- added D9: SMAZ24-13-F, USBPOWER45:D_SMA, symbol USBPOWER45:D_Zener
- added Q2: BCX53-16,115, USBPOWER45:SOT-89-3, symbol USBPOWER45:BCX53_NXP
- added Q3: MMBT3906, USBPOWER45:SOT-23, symbol USBPOWER45:MMBT3906
- added R23: 33, USBPOWER45:R_0603_1608Metric, symbol USBPOWER45:R
- added R24: 6.8k, USBPOWER45:R_0603_1608Metric, symbol USBPOWER45:R
- added R25: 100k, USBPOWER45:R_0603_1608Metric, symbol USBPOWER45:R
- added R26: 20k, USBPOWER45:R_0603_1608Metric, symbol USBPOWER45:R
- added R27: 10k, USBPOWER45:R_1206_3216Metric, symbol USBPOWER45:R
- added R28: 10k, USBPOWER45:R_0603_1608Metric, symbol USBPOWER45:R
- added R29: 1k, USBPOWER45:R_0603_1608Metric, symbol USBPOWER45:R
- added TP1: VPD, USBPOWER45:TestPoint_Pad_D1.0mm, symbol USBPOWER45:TestPoint
- added TP2: VPD_U1, USBPOWER45:TestPoint_Pad_D1.0mm, symbol USBPOWER45:TestPoint
- added TP3: EF_IN, USBPOWER45:TestPoint_Pad_D1.0mm, symbol USBPOWER45:TestPoint
- added TP4: VIN, USBPOWER45:TestPoint_Pad_D1.0mm, symbol USBPOWER45:TestPoint
- added TP5: EN_P, USBPOWER45:TestPoint_Pad_D1.0mm, symbol USBPOWER45:TestPoint
- added TP6: EF_FLT, USBPOWER45:TestPoint_Pad_D1.0mm, symbol USBPOWER45:TestPoint
- added TP7: EF_IMON, USBPOWER45:TestPoint_Pad_D1.0mm, symbol USBPOWER45:TestPoint
- added TP8: GND, USBPOWER45:TestPoint_Pad_D1.0mm, symbol USBPOWER45:TestPoint
- C1: Note CH224A VHV decoupling -> At U1 VHV/VBUS; after Q2
- C2: Note U5 IN cap. C1 + C2 = all the capacitance VBUS sees at attac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 -> U5 IN/P_IN local cap. With C1, approximately 2 uF at attach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
- C3: value 1n -> 22n; LCSC C1588 -> C21122; MPN CL10B102KB8NNNC -> CL10B223KB8NNNC; Note dVdt: 2000 / 1000 pF = 2 V/ms, VIN 0 -> 20 V in ~10 ms, ~0.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 -> dVdt: 2 uA x 25 / 22 nF = 2.27 V/ms; ~9 ms ramp, followed b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
- C5: Note Aluminium bulk on VIN, behind the eFuse: damps the converte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 -> Bulk behind U5; input damping
- D1: value SMBJ20A -> SMBJ22A; LCSC C10213 -> C10214; MPN SMBJ20A -> SMBJ22A; Note Unidirectional TVS, 20 V stand-off / 22.2 V min breakdown (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 -> 22 V stand-off, 35.5 V rated clamp at 16.9 A (10/1000 us), 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
- F1: value 5A -> 5A 63V; LCSC C57525 -> C553937; MPN 0466005.NRHF -> S1206-SD-5.0A; Manufacturer Littelfuse -> SART(Nanjing Sart Tech); Note 5 A fast 1206 fuse (32 V class): back-up only, U5 limits at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 -> 63 V DC, 50 A interrupt rating. Backup fuse, NOT the USB cu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
- R1: Note CH224A CFG1 to GND: 120k = 20 V request -> CFG1: 120k = 20 V request
- R2: Note UVLO/OVLO divider: on >= 1.2 x 107.3/7.3 = 17.6 V, off < 16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 -> UVLO top: qualified-source voltage sensed before D10
- R3: value 2.2k -> 7.5k; LCSC C4190 -> C23234; MPN 0603WAF2201T5E -> 0603WAF7501T5E; Note UVLO/OVLO divider, see R2 -> UVLO on 17.20 V / off 16.08 V nominal; tolerance/leakage co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
- R4: value 5.1k -> 120k; LCSC C23186 -> C25808; MPN 0603WAF5101T5E -> 0603WAF1203T5E; Note UVLO/OVLO divider: OVLO cuts VIN above 1.2 x 107.3/5.1 = 25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 -> OVP top with R28; independent of UVLO and RESET
- R5: value 820 -> 3.3k; LCSC C23253 -> C22978; MPN 0603WAF8200T5E -> 0603WAF3301T5E; Note ILM: limit 3334 / 820 = 4.1 A (+/-10 %) -> Series R5 + R29 = 4.3k: 4.186 A nominal. +/-10% IC and R to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
- R6: Note EN_P = VIN / 11 = 1.8 V at 20 V (TPS62933 EN max 5.5 V, AUX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 -> Safe EN divider + U5 PGOOD open drain. Fault turnoff has 8-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
- R7: Note EN_P divider bottom, see R6 -> EN_P = VIN/11 while PGOOD is released
- SW1: Note RESET, as usb-power SW1 (P021301 Rev B: contacts 1+3 common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 -> RESET: press grounds U5 SHDN (internally pulled up to 2.7 V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
- U1: Note USB PD sink, fixed 20 V request (CFG1 120k). Powered from V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 -> Fixed 20 V request, independently current-limited/zener-pro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
- U5: value TPS259470ARPWR -> TPS16630PWPR; footprint USBPOWER45:Texas_RPW0010A_VQFN-HR-10_2x2mm_P0.45mm -> USBPOWER45:HTSSOP-20-1EP_4.4x6.5mm_P0.65mm_EP3.4x6.5mm_Mask2.96x2.96mm_ThermalVias; symbol USBPOWER45:TPS259470ARPW -> USBPOWER45:TPS16630PWP; LCSC C3662799 -> C1849461; MPN TPS259470ARPWR -> TPS16630PWPR; Note eFuse (SLVSFC9C): 2.7-23 V, 28 mOhm, OVLO, active current l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 -> 60 V eFuse, 31 mOhm typ; 4.19 A nominal limit, auto-retry, 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
Connections:
- net EF_TMR is gone; now on net EF_DVDT: U5.10 (dVdT)
- net EF_DVDT: no longer U5.7 (DVDT)
- net EF_ILM: now also U5.11 (ILIM); no longer U5.9 (ILM)
- net EF_OV: now also R4.2, U5.8 (OVP), R24.1; no longer R3.2, R4.1, U5.2 (OVLO)
- net EF_UV: now also U5.7 (UVLO); no longer SW1.1 (COMMON), SW1.3 (COMMON), U5.1 (EN/UVLO)
- net EN_P: now also U5.16 (PGOOD), TP5.1; no longer U5.3 (AUXOFF)
- net GND: now also R3.2, U5.12 (MODE), U5.21 (EP), U5.9 (GND), D9.2 (A), R24.2, R26.2, R27.2, R29.2, TP8.1; no longer R4.2, R5.2, U5.8 (GND)
- net VIN: now also U5.18 (OUT), U5.19 (OUT), U5.20 (OUT), TP4.1; no longer U5.6 (OUT)
- net VPD: now also D10.2 (A), D11.1 (K), Q3.2 (E), R23.1, R25.1, R28.1, TP1.1; no longer C1.1, C2.1, U1.1 (VHV), U1.8 (VBUS_SENSE), U5.5 (IN)
- new net: R28.2, R4.1
- new net: R29.1, R5.2
- new net EF_FLT: R25.2, TP6.1, U5.15 (~{FLT})
- new net EF_IMON: R26.1, TP7.1, U5.14 (IMON)
- new net EF_IN: C2.1, D10.1 (K), TP3.1, U5.1 (IN), U5.2 (IN), U5.3 (IN), U5.6 (P_IN)
- new net EF_SHDN: SW1.1 (COMMON), SW1.3 (COMMON), U5.13 (~{SHDN})
- new net PD_BASE: Q2.3 (B), Q3.3 (C), R27.1
- new net PD_SENSE: Q2.1 (E), Q3.1 (B), R23.2
- new net VPD_U1: C1.1, D11.2 (A), D9.1 (K), Q2.2 (C), TP2.1, U1.1 (VHV), U1.8 (VBUS_SENSE)
- no-connect marks 20 -> 22
Other:
- note added: "+12V: TPS62933F, forced PWM, 1.2 MHz, 6.8 uH"
- note added: "+5V: TPS62933F, forced PWM, ~2.0 MHz, 3.3 uH"
- note added: "-12V: LMR38020F inverting buck-boost, forced PWM, ~790 kHz, 15 uH. IC ground = -12V."
- note added: "Board limit: 4.3k = 3.3k + 1k; screened USB steady limit <=4.724 A. Full-load estimate ~66 W input, not a rating."
- note added: "Bulk caps, polarity clamps and rail LEDs (unchanged)"
- note added: "D10 upgraded to 10 A SMC; thermal copper required. Smaller sources may trip/cycle. Test thermal / PD / surge / startup."
- note added: "No guaranteed discharge time / complete module reset"
- note added: "OUTPUTS: parallel 16-pin Eurorack headers (pin 1 = -12V). Not for paralleling independent supplies."
- note added: "PANEL: SW1 input disable/restart; D8 +5V presence"
- note added: "S5 INPUT: USB PD 20 V; 5 A contract/cable for full load. Board eFuse limit 4.19 A; no adapter-power tracking."
- note added: "TARGETS: +12V 2.5 A / +5V 2.5 A / -12V 1.0 A = 54.5 W total; simultaneous operation needs bench qualification."
- note added: "TP5 = EN_P; TP6 = raw-voltage FLT; TP7 = 0.558 V/A typical; TP8 = system GND. D10 blocks USB backfeed."
- note added: "U1 ONLY: Q2/Q3 + R23 current limiter (~18 mA typ) feeds a 24 V shunt. Verify U1 <30 V."
- note added: "U5 TPS16630: 60 V input; UVLO 17.2 V / OVP 24.14 V nominal; ~9 ms ramp + PGOOD delay; auto-retry."
- note added: "UVLO / OVP / ramp / current / enable / diagnostic networks"
- note added: "Unchanged divider: 0.8 x (1 + 47k/3.3k) = 12.19 V nominal"
- note added: "Unchanged divider: 0.8 x (1 + 68k/13k) = 4.98 V nominal"
- note added: "Unchanged power stage. Q1 enables from +12V, not a precision all-rail supervisor. Validate loop stability."
- note removed: "+12V: U2 TPS62933F, forced PWM, 1.2 MHz, 6.8 uH. VOUT = 0.8 V x (1 + 47k / 3.3k) = 12.19 V"
- note removed: "+5V: U3 TPS62933F, forced PWM, ~2.0 MHz (RT 10k), 3.3 uH. VOUT = 0.8 V x (1 + 68k / 13k) = 4.98 V"
- note removed: "-12V: U4 LMR38020F inverting buck-boost, forced PWM, ~790 kHz (RT 33k), 15 uH. IC ground pins = -12V. |VOUT| = 1.0 V x (1 + 100k / 9.1k) = 11.99 V"
- note removed: "Budget (docs/design.md): +12V 2.5 A, +5V 2.5 A, -12V 1.0 A per rail; all rails together <= ~39 W out on a 45 W charger (~52 W on 60 W)"
- note removed: "Bulk caps, rail clamps (SS34) and rail LEDs at the headers"
- note removed: "FRONT PANEL (as usb-power): SW1 RESET pulls U5 EN/UVLO low: all rails off,"
- note removed: "OUTPUT: 2 x 16-pin Eurorack box header in parallel (Doepfer pinout, pin 1 = -12V)"
- note removed: "Q1: -12V is enabled from +12V (starts at +12V ~ 8 V, stops when +12V goes): the -12V rail never runs alone. Internal compensation"
- note removed: "U5 TPS259470A eFuse: on 17.6-25.3 V only (R2/R3/R4), VIN ramps at 2 V/ms (C3), limit 4.1 A (R5), auto-retry. AUXOFF holds EN_P low until VIN has ramped, then U2/U3 start"
- note removed: "USB-C PD 20 V INPUT: CH224A (CFG1 120k = 20 V), 5 A fuse, SMBJ20A TVS. VBUS sees only C1 + C2 (2 uF) at attach. Use a 20 V PD charger rated 45 W or more; 60 W for the full budget"
- note removed: "release = restart. D8 red 3 mm +5V power LED (hand-soldered)"
- moved on the sheet: C1, C10, C11, C12, C13, C14, C15, C16, C17, C18, C19, C2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

Commit message: Improve the 45w usb power module.
Parts:
- removed C1, C2: 1u, USBPOWER45:C_0603_1608Metric, symbol USBPOWER45:C
- removed C10, C17, C19, C27, C28, C8: 100n, USBPOWER45:C_0603_1608Metric, symbol USBPOWER45:C
- removed C11, C12, C13, C14, C20, C21, C22, C23, C29, C30, C31, C32, C33: 22u, USBPOWER45:C_1206_3216Metric, symbol USBPOWER45:C
- removed C15, C16, C24, C25, C26, C6, C7: 10u, USBPOWER45:C_1206_3216Metric, symbol USBPOWER45:C
- removed C18, C3, C9: 22n, USBPOWER45:C_0603_1608Metric, symbol USBPOWER45:C
- removed C34, C35, C36: 100u, USBPOWER45:CP_Elec_6.3x7.7, symbol USBPOWER45:C_Polarized
- removed C5: 47u, USBPOWER45:CP_Elec_6.3x7.7, symbol USBPOWER45:C_Polarized
- removed D1: SMBJ22A, USBPOWER45:D_SMB, symbol USBPOWER45:D_Zener
- removed D10: SS1060, USBPOWER45:D_SMC, symbol USBPOWER45:D_Schottky
- removed D11, D2, D3, D4: SS34, USBPOWER45:D_SMA, symbol USBPOWER45:D_Schottky
- removed D5, D6, D7: RED, USBPOWER45:LED_0603_1608Metric, symbol USBPOWER45:LED
- removed D8: RED 3mm, USBPOWER45:LED_D3.0mm_Horizontal_O1.27mm_Z2.0mm_Edge, symbol USBPOWER45:LED
- removed D9: SMAZ24-13-F, USBPOWER45:D_SMA, symbol USBPOWER45:D_Zener
- removed F1: 5A 63V, USBPOWER45:Fuse_1206_3216Metric, symbol USBPOWER45:Fuse
- removed J1: TYPE-C-31-M-12, USBPOWER45:HRO-TYPE-C-31-M-12, symbol USBPOWER45:HRO_TYPE_C_31_M_12
- removed J2, J3: IDC 2x8 box header, USBPOWER45:IDC-Header_2x08_P2.54mm_Vertical, symbol USBPOWER45:Conn_02x08_Odd_Even
- removed L1: 6.8u, USBPOWER45:L_SLO1040H6R8MTT, symbol USBPOWER45:L
- removed L2: 3.3u, USBPOWER45:L_SLO1040H6R8MTT, symbol USBPOWER45:L
- removed L3: 15u, USBPOWER45:L_SLO1040H6R8MTT, symbol USBPOWER45:L
- removed Q1, Q3: MMBT3906, USBPOWER45:SOT-23, symbol USBPOWER45:MMBT3906
- removed Q2: BCX53-16,115, USBPOWER45:SOT-89-3, symbol USBPOWER45:BCX53_NXP
- removed R1, R4: 120k, USBPOWER45:R_0603_1608Metric, symbol USBPOWER45:R
- removed R10, R19, R21, R28, R7: 10k, USBPOWER45:R_0603_1608Metric, symbol USBPOWER45:R
- removed R11: 68k, USBPOWER45:R_0603_1608Metric, symbol USBPOWER45:R
- removed R12: 13k, USBPOWER45:R_0603_1608Metric, symbol USBPOWER45:R
- removed R13: 33k, USBPOWER45:R_0603_1608Metric, symbol USBPOWER45:R
- removed R14, R16, R17, R2, R25, R6: 100k, USBPOWER45:R_0603_1608Metric, symbol USBPOWER45:R
- removed R15: 9.1k, USBPOWER45:R_0603_1608Metric, symbol USBPOWER45:R
- removed R18, R26: 20k, USBPOWER45:R_0603_1608Metric, symbol USBPOWER45:R
- removed R20, R22, R29: 1k, USBPOWER45:R_0603_1608Metric, symbol USBPOWER45:R
- removed R23: 33, USBPOWER45:R_0603_1608Metric, symbol USBPOWER45:R
- removed R24: 6.8k, USBPOWER45:R_0603_1608Metric, symbol USBPOWER45:R
- removed R27: 10k, USBPOWER45:R_1206_3216Metric, symbol USBPOWER45:R
- removed R3: 7.5k, USBPOWER45:R_0603_1608Metric, symbol USBPOWER45:R
- removed R5, R9: 3.3k, USBPOWER45:R_0603_1608Metric, symbol USBPOWER45:R
- removed R8: 47k, USBPOWER45:R_0603_1608Metric, symbol USBPOWER45:R
- removed SW1: TL3340AF160QG, USBPOWER45:SW_TL3340AF160QG_HandSolder, symbol USBPOWER45:TL3340AF160QG
- removed TP1: VPD, USBPOWER45:TestPoint_Pad_D1.0mm, symbol USBPOWER45:TestPoint
- removed TP2: VPD_U1, USBPOWER45:TestPoint_Pad_D1.0mm, symbol USBPOWER45:TestPoint
- removed TP3: EF_IN, USBPOWER45:TestPoint_Pad_D1.0mm, symbol USBPOWER45:TestPoint
- removed TP4: VIN, USBPOWER45:TestPoint_Pad_D1.0mm, symbol USBPOWER45:TestPoint
- removed TP5: EN_P, USBPOWER45:TestPoint_Pad_D1.0mm, symbol USBPOWER45:TestPoint
- removed TP6: EF_FLT, USBPOWER45:TestPoint_Pad_D1.0mm, symbol USBPOWER45:TestPoint
- removed TP7: EF_IMON, USBPOWER45:TestPoint_Pad_D1.0mm, symbol USBPOWER45:TestPoint
- removed TP8: GND, USBPOWER45:TestPoint_Pad_D1.0mm, symbol USBPOWER45:TestPoint
- removed U1: CH224A, USBPOWER45:SSOP-10-1EP_3.9x4.9mm_P1mm_EP2.1x3.3mm, symbol USBPOWER45:CH224A
- removed U2, U3: TPS62933FDRLR, USBPOWER45:SOT-583-8, symbol USBPOWER45:TPS62933F
- removed U4: LMR38020FDDAR, USBPOWER45:TI_SO-PowerPAD-8_ThermalVias, symbol USBPOWER45:LMR38020FDDA
- removed U5: TPS16630PWPR, USBPOWER45:HTSSOP-20-1EP_4.4x6.5mm_P0.65mm_EP3.4x6.5mm_Mask2.96x2.96mm_ThermalVias, symbol USBPOWER45:TPS16630PWP
Connections:
- no-connect marks 22 -> 0
Other:
- added sheet +12 V converter and output eFuse (02_positive_12v.kicad_sch)
- added sheet +5 V converter and output eFuse (03_positive_5v.kicad_sch)
- added sheet Always-on control - all-rail fault latch and RESET (06_fault_reset.kicad_sch)
- added sheet Negative converter - raw rail (04_negative_converter.kicad_sch)
- added sheet Negative rail protection and level shifting (05_negative_protection.kicad_sch)
- added sheet Protected outputs - voltage monitors and panel LEDs (07_outputs_status.kicad_sch)
- added sheet USB PD and main eFuse (01_usb_input.kicad_sch)
- note added: "60 V always-on LDO / retained ARMED + FAULT Manual RESET disables all three rails"
- note added: "CH224A: 20 V request TPS16630: 4.186 A nominal"
- note added: "FAULT POLICY Each rail detects independently. Persistent fault -> all OFF until RESET. Main LED is not merely a +5 V lamp."
- note added: "LM5067 + external N-MOSFET 1.0 A nominal / optical control"
- note added: "LMR38020F inverting buck-boost RAW negative supply"
- note added: "OUTPUTS: +12 / +5 / -12 Nominal limits: 2.647 / 2.647 / 1.0 A Tolerance and thermal limits apply. Not a guaranteed 54.5 W simultaneous rating."
- note added: "Parallel Eurorack headers MAIN, +12, +5 and -12 LEDs"
- note added: "S6 schematic only. All three converters retained; main and + rails TPS16630; negative LM5067 + MOSFET."
- note added: "TPS62933F -> TPS16630 +12 V protected output"
- note added: "TPS62933F -> TPS16630 +5 V protected output"
- note added: "USB POWER / ALL-RAIL PROTECTION AND RESET"
- note removed: "+12V: TPS62933F, forced PWM, 1.2 MHz, 6.8 uH"
- note removed: "+5V: TPS62933F, forced PWM, ~2.0 MHz, 3.3 uH"
- note removed: "-12V: LMR38020F inverting buck-boost, forced PWM, ~790 kHz, 15 uH. IC ground = -12V."
- note removed: "Board limit: 4.3k = 3.3k + 1k; screened USB steady limit <=4.724 A. Full-load estimate ~66 W input, not a rating."
- note removed: "Bulk caps, polarity clamps and rail LEDs (unchanged)"
- note removed: "D10 upgraded to 10 A SMC; thermal copper required. Smaller sources may trip/cycle. Test thermal / PD / surge / startup."
- note removed: "No guaranteed discharge time / complete module reset"
- note removed: "OUTPUTS: parallel 16-pin Eurorack headers (pin 1 = -12V). Not for paralleling independent supplies."
- note removed: "PANEL: SW1 input disable/restart; D8 +5V presence"
- note removed: "S5 INPUT: USB PD 20 V; 5 A contract/cable for full load. Board eFuse limit 4.19 A; no adapter-power tracking."
- note removed: "TARGETS: +12V 2.5 A / +5V 2.5 A / -12V 1.0 A = 54.5 W total; simultaneous operation needs bench qualification."
- note removed: "TP5 = EN_P; TP6 = raw-voltage FLT; TP7 = 0.558 V/A typical; TP8 = system GND. D10 blocks USB backfeed."
- note removed: "U1 ONLY: Q2/Q3 + R23 current limiter (~18 mA typ) feeds a 24 V shunt. Verify U1 <30 V."
- note removed: "U5 TPS16630: 60 V input; UVLO 17.2 V / OVP 24.14 V nominal; ~9 ms ramp + PGOOD delay; auto-retry."
- note removed: "UVLO / OVP / ramp / current / enable / diagnostic networks"
- note removed: "Unchanged divider: 0.8 x (1 + 47k/3.3k) = 12.19 V nominal"
- note removed: "Unchanged divider: 0.8 x (1 + 68k/13k) = 4.98 V nominal"
- note removed: "Unchanged power stage. Q1 enables from +12V, not a precision all-rail supervisor. Validate loop stability."
- title: Big Modular - usb-power-45w -> USB power - wired power flow and protection overview
